File: KiCAD/OsmoFresh_Quella_PRO/mainpcb.connectors.kicad_sch (KiCad schematic)
At the start: 14 parts, among them CN1 Conn_01x02_Pin, CN10 Conn_01x06_Pin, CN11 Conn_01x04_Pin, CN12 Conn_01x02_Pin, CN13 Conn_01x02_Pin, CN14 Conn_01x02_Pin, CN16 Conn_01x02_Pin, CN2 Conn_01x02_Pin, CN3 Conn_01x02_Pin, CN5 Conn_01x02_Pin, CN6 Conn_01x02_Pin, CN7 Conn_01x02_Pin, CN8 Conn_01x02_Pin, CN9 Conn_01x02_Pin

Commit message: Update Schematics
Connections:
- net Internal_Tank_Level_Black+: now also CN6.2 (Pin_2); no longer CN6.1 (Pin_1)
- net Internal_Tank_Level_Black-: now also CN6.1 (Pin_1); no longer CN6.2 (Pin_2)
- net Internal_Tank_Level_Red+: now also CN14.2 (Pin_2); no longer CN14.1 (Pin_1)
- net Internal_Tank_Level_Red-: now also CN14.1 (Pin_1); no longer CN14.2 (Pin_2)
Changed lines of the file:
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@@
+	(wire
+		(pts
+			(xy 143.51 93.98) (xy 146.05 93.98)
+		)
+		(stroke
+			(width 0)
+			(type default)
+		)
+	)
+	(wire
+		(pts
+			(xy 143.51 119.38) (xy 146.05 119.38)
+		)
+		(stroke
+			(width 0)
+			(type default)
+		)
+	)
+	(wire
+		(pts
+			(xy 143.51 101.6) (xy 146.05 101.6)
+		)
+		(stroke
+			(width 0)
+			(type default)
+		)
+	)
+	(wire
+		(pts
+			(xy 143.51 109.22) (xy 146.05 109.22)
+		)
+		(stroke
+			(width 0)
+			(type default)
+		)
+	)
+	(wire
+		(pts
+			(xy 143.51 55.88) (xy 146.05 55.88)
+		)
+		(stroke
+			(width 0)
+			(type default)
+		)
+	)
+	(wire
+		(pts
+			(xy 143.51 130.81) (xy 146.05 130.81)
+		)
+		(stroke
+			(width 0)
+			(type default)
+		)
+	)
+	(wire
+		(pts
+			(xy 143.51 50.8) (xy 146.05 50.8)
+		)
+		(stroke
+			(width 0)
+			(type default)
+		)
+	)
+	(wire
+		(pts
+			(xy 143.51 127) (xy 146.05 127)
+		)
+		(stroke
+			(width 0)
+			(type default)
+		)
+	)
+	(wire
+		(pts
+			(xy 143.51 58.42) (xy 146.05 58.42)
+		)
+		(stroke
+			(width 0)
+			(type default)
+		)
+	)
+	(wire
+		(pts
+			(xy 143.51 151.13) (xy 146.05 151.13)
+		)
+		(stroke
+			(width 0)
+			(type default)
+		)
+	)
+	(wire
+		(pts
+			(xy 143.51 124.46) (xy 146.05 124.46)
+		)
+		(stroke
+			(width 0)
+			(type default)
+		)
+	)
+	(wire
+		(pts
+			(xy 143.51 88.9) (xy 146.05 88.9)
+		)
+		(stroke
+			(width 0)
+			(type default)
+		)
+	)
+	(wire
+		(pts
+			(xy 143.51 40.64) (xy 146.05 40.64)
+		)
+		(stroke
+			(width 0)
+			(type default)
+		)
+	)
+	(wire
+		(pts
+			(xy 143.51 71.12) (xy 146.05 71.12)
+		)
+		(stroke
+			(width 0)
+			(type default)
+		)
+	)
+	(wire
+		(pts
+			(xy 143.51 48.26) (xy 146.05 48.26)
+		)
+		(stroke
+			(width 0)
+			(type default)
+		)
+	)
 	(wire
 		(pts
@@
 	(wire
 		(pts
-			(xy 143.51 93.98) (xy 146.05 93.98)
-		)
-		(stroke
-			(width 0)
-			(type default)
-		)
-	)
-	(wire
-		(pts
-			(xy 143.51 119.38) (xy 146.05 119.38)
-		)
-		(stroke
-			(width 0)
-			(type default)
-		)
-	)
-	(wire
-		(pts
-			(xy 143.51 109.22) (xy 146.05 109.22)
-		)
-		(stroke
-			(width 0)
-			(type default)
-		)
-	)
-	(wire
-		(pts
-			(xy 143.51 55.88) (xy 146.05 55.88)
-		)
-		(stroke
-			(width 0)
-			(type default)
-		)
-	)
-	(wire
-		(pts
-			(xy 143.51 130.81) (xy 146.05 130.81)
-		)
-		(stroke
-			(width 0)
-			(type default)
-		)
-	)
-	(wire
-		(pts
-			(xy 143.51 50.8) (xy 146.05 50.8)
-		)
-		(stroke
-			(width 0)
-			(type default)
-		)
-	)
-	(wire
-		(pts
-			(xy 143.51 127) (xy 146.05 127)
-		)
-		(stroke
-			(width 0)
-			(type default)
-		)
-	)
-	(wire
-		(pts
-			(xy 143.51 58.42) (xy 146.05 58.42)
-		)
-		(stroke
-			(width 0)
-			(type default)
-		)
-	)
-	(wire
-		(pts
-			(xy 143.51 151.13) (xy 146.05 151.13)
-		)
-		(stroke
-			(width 0)
-			(type default)
-		)
-	)
-	(wire
-		(pts
-			(xy 143.51 124.46) (xy 146.05 124.46)
-		)
-		(stroke
-			(width 0)
-			(type default)
-		)
-	)
-	(wire
-		(pts
-			(xy 143.51 88.9) (xy 146.05 88.9)
-		)
-		(stroke
-			(width 0)
-			(type default)
-		)
-	)
-	(wire
-		(pts
-			(xy 143.51 40.64) (xy 146.05 40.64)
-		)
-		(stroke
-			(width 0)
-			(type default)
-		)
-	)
-	(wire
-		(pts
-			(xy 143.51 71.12) (xy 146.05 71.12)
-		)
-		(stroke
-			(width 0)
-			(type default)
-		)
-	)
-	(wire
-		(pts
-			(xy 143.51 48.26) (xy 146.05 48.26)
-		)
-		(stroke
-			(width 0)
-			(type default)
-		)
-	)
-	(wire
-		(pts
 			(xy 143.51 43.18) (xy 146.05 43.18)
 		)
@@
 		(pts
 			(xy 143.51 38.1) (xy 146.05 38.1)
-		)
-		(stroke
-			(width 0)
-			(type default)
-		)
-	)
-	(wire
-		(pts
-			(xy 143.51 101.6) (xy 146.05 101.6)
 		)
 		(stroke
@@
 	)
 	(global_label "Internal_Tank_Level_Red-"
-		(shape output)
-		(at 146.05 104.14 0)
-		(fields_autoplaced yes)
-		(effects
-			(font
-				(size 1.27 1.27)
-			)
-			(justify left)
-		)
-		(property "Intersheetrefs" "${INTERSHEET_REFS}"
-			(at 173.4673 104.14 0)
+		(shape input)
+		(at 146.05 101.6 0)
+		(fields_autoplaced yes)
+		(effects
+			(font
+				(size 1.27 1.27)
+			)
+			(justify left)
+		)
+		(property "Intersheetrefs" "${INTERSHEET_REFS}"
+			(at 173.4673 101.6 0)
 			(hide yes)
 			(show_name no)
@@
 		)
 	)
-	(global_label "Internal_Tank_Level_Black-"
+	(global_label "Internal_Tank_Level_Black+"
 		(shape output)
 		(at 146.05 111.76 0)
@@
 	(global_label "Internal_Tank_Level_Red+"
 		(shape output)
-		(at 146.05 101.6 0)
-		(fields_autoplaced yes)
-		(effects
-			(font
-				(size 1.27 1.27)
-			)
-			(justify left)
-		)
-		(property "Intersheetrefs" "${INTERSHEET_REFS}"
-			(at 173.4673 101.6 0)
+		(at 146.05 104.14 0)
+		(fields_autoplaced yes)
+		(effects
+			(font
+				(size 1.27 1.27)
+			)
+			(justify left)
+		)
+		(property "Intersheetrefs" "${INTERSHEET_REFS}"
+			(at 173.4673 104.14 0)
 			(hide yes)
 			(show_name no)
@@
 		)
 	)
-	(global_label "Internal_Tank_Level_Black+"
-		(shape output)
+	(global_label "Internal_Tank_Level_Black-"
+		(shape input)
 		(at 146.05 109.22 0)
 		(fields_autoplaced yes)

Commit message: Update Schematics
Changed lines of the file:
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@@
 	)
 	(global_label "TDS-"
-		(shape output)
+		(shape input)
 		(at 146.05 81.28 0)
 		(fields_autoplaced yes)
@@
 	)
 	(global_label "Temperature_Outlet-"
-		(shape output)
+		(shape input)
 		(at 146.05 58.42 0)
 		(fields_autoplaced yes)
@@
 	)
 	(global_label "UNUSED_CN8-"
-		(shape bidirectional)
+		(shape input)
 		(at 146.05 73.66 0)
 		(fields_autoplaced yes)
@@
 		)
 		(property "Intersheetrefs" "${INTERSHEET_REFS}"
-			(at 164.1165 73.66 0)
+			(at 163.0052 73.66 0)
 			(hide yes)
 			(show_name no)
@@
 	)
 	(global_label "Water_Tank_Empty-"
-		(shape output)
+		(shape input)
 		(at 146.05 96.52 0)
 		(fields_autoplaced yes)
@@
 	)
 	(global_label "UNUSED_CN8+"
-		(shape bidirectional)
+		(shape output)
 		(at 146.05 71.12 0)
 		(fields_autoplaced yes)
@@
 		)
 		(property "Intersheetrefs" "${INTERSHEET_REFS}"
-			(at 164.1165 71.12 0)
-			(hide yes)
-			(show_name no)
+			(at 163.0052 71.12 0)
+			(hide yes)
+			(show_name no)
