File: KiCAD/OsmoFresh_Quella_PRO/mainpcb.secondary.kicad_sch (KiCad schematic)
At the start: 7 parts, among them K2 [NO]

Commit message: Update Schematics
Parts:
- removed T2: (no value), symbol Device:Transformer_1P_1S
- added C1: (no value), symbol Device:C
- added C?: 470µF 50V, symbol Device:C_Polarized
- added D5: D, symbol Device:D
- added Q2: (no value), symbol Transistor_FET:Q_NMOS_DGS
- added R15: 10kΩ, symbol Device:R
- added R17: 2kΩ, symbol Device:R
- added R30, R35, R37: 20kΩ, symbol Device:R
- added R62, R63: 0,62Ω, symbol Device:R
- added U4: ULN2003A, symbol Transistor_Array:ULN2003A
- C11: value C -> unkown
- K2: value [NO] -> 5A 250Vac
Connections:
- net Current_Sense+: now reaches C11.2, R32.2, R33.2
- net at K2.A1: no longer D5.1 (K)
- net at K2.A2: no longer D5.2 (A)
- net Current_Sense-: now reaches C11.1, R31.1, R32.1
- net +24Vdc: now reaches K2.13
- net +24Vdc: now also D5.1 (K), C1.1, C?.1, U4.9 (COM)
- net Water_Pump+: now reaches K2.14
- net Water_Pump+: now also D5.1 (K)
- new net: Q2.2 (G), R15.1, R17.2
- new net Flush_Valve-: U4.10 (O7), U4.11 (O6), U4.12 (O5)
- new net GND: C1.2, C?.2, Q2.3 (S), R15.2, R62.1, R63.2, U4.8 (GND)
- new net IC1_Pin5: R30.1, U4.5 (I5), U4.6 (I6), U4.7 (I7)
- new net IC1_Pin6: R35.1, U4.2 (I2), U4.3 (I3), U4.4 (I4)
- new net IC1_Pin7: R37.1, U4.1 (I1)
- new net Relay_Heater_1200W (IC1_Pin2): R17.1
- new net Relay_Heater_Coil-: D5.2 (A), Q2.1 (D)
- new net UNUSED_CN10-: U4.13 (O4), U4.14 (O3), U4.15 (O2)
- new net UNUSED_CN13-: U4.16 (O1)
- new net Water_Pump-: D5.2 (A), R30.2, R35.2, R37.2, R62.2, R63.1
Other:
- note added: "Vuanze Electric Y32F-SS-124DM"
- title: MainPCB.Secondary -> MainPCB Secondary
- moved on the sheet: C11, D5, R31, R32, R33

Commit message: Update Filestructure
Parts:
- added C11, C3, C6: C, symbol Device:C
- added R22, R45, R64: 2kΩ, symbol Device:R
Connections:
- net Water_Pump-: now also R64.1
- new net: C3.1, R45.2
- new net: C6.1, R64.2
- new net: C11.1, C6.2
- new net: C11.2, R22.1
- new net: R22.2, R45.1
Other:
- moved on the sheet: R30, R35, R37, U4

Commit message: Update Schematics
Parts:
- removed R31, R33: 10 kΩ, symbol Device:R
- removed R32: 1 kΩ, symbol Device:R
- added C27, C4: unkown, symbol Device:C
- added R25: 1kΩ, symbol Device:R
- added R29, R30, R40 (x2), R6: 10kΩ, symbol Device:R
- added R5: 2kΩ, symbol Device:R
- renumbered C11 to C10, R30 to R36
Connections:
- net Current_Sense+: now also R22.2, R45.1, R25.1, R30.2
- net Current_Sense-: now also R25.2, R29.2
- net GND: now also C27.1
- net at C3.2: now also C4.1, R29.1, R40.1, R6.2
- new net: C27.2, R40.1, R40.2
- new net: R30.1, R40.2
- new net IC1_Pin10: C4.2, R5.2
- new net Temperature_Outlet+: R5.1, R6.1
Other:
- note added: "1"
- note added: "2"
- note added: "3"
- note added: "4"
- note added: "5"
- note added: "6"
- note added: "7"
- note added: "8"
- note added: "U5 KM393"
- moved on the sheet: C10, C3

Commit message: Update Schematics
Parts:
- removed Q2: (no value), symbol Transistor_FET:Q_NMOS_DGS
- added C12, C13, C14, C15, C16, C17, C18, C19, C2, C20, C21, C22, C23, C24, C25, C26, C5, C7, C8, C9: unkown, symbol Device:C
- added D6, D7: D, symbol Device:D
- added EC2: 30µF 10V, symbol Device:C_Polarized
- added L1: (no value), symbol Device:L
- added Q2: NMOS, symbol Simulation_SPICE:NMOS
- added Q3, Q5, Q6, Q8: NPN, symbol Simulation_SPICE:NPN
- added Q4: PMOS, symbol Simulation_SPICE:PMOS
- added R10, R12, R13, R24, R4, R65, R66: 2kΩ, symbol Device:R
- added R11, R20, R33, R53, R54, R60, R67, R68: 10kΩ, symbol Device:R
- added R14, R16, R21: 1kΩ, symbol Device:R
- added R18, R31: 4,7kΩ, symbol Device:R
- added R19, R59: 470Ω, symbol Device:R
- added R23, R61: 47kΩ, symbol Device:R
- added R32: 5,1kΩ, symbol Device:R
- added R34: 510Ω, symbol Device:R
- added R44: 330Ω, symbol Device:R
- added R49, R50: 220Ω, symbol Device:R
- added R51, R52: 750Ω, symbol Device:R
- added R55: 5,1Ω, symbol Device:R
- added RL1: Ω, symbol Device:R
- gave numbers to parts that had none: 1
- renumbered D5 to D4, R40 to R41
Connections:
- net +24Vdc: now also Q4.3 (S), R51.2
- net GND: now also Q2.1 (D), R55.1
- net IC1_Pin6: now also C11.1, C6.2
- net Relay_Heater_Coil-: now also Q2.2 (G)
- net at R15.1, R17.2: now also Q2.3 (S)
- net U3 Vin: now reaches R30.1, R41.2
- net Q8_Emitter: now reaches C6.1, R64.2
- net Q8_Emitter: now also Q8.3 (E)
- net IC1_Pin12: now reaches C11.2, R22.1
- net Current_Sense+ renamed Transformer+
- net Current_Sense- renamed Transformer-
- new net: Q4.2 (G), R51.1, R52.2
- new net: C18.2, C19.1
- new net: C19.2, R53.2, R54.1
- new net: Q8.1 (C), R52.1
- new net: R32.2, R33.1
- new net: Q8.2 (B), R33.2
- new net IC1_Pin15: C18.1, R54.2
- new net IC1_Pin17: R12.1
- new net IC1_Pin18: R13.1
- new net IC1_Pin3: R32.1
- new net Internal_Tank_Level_Black+: R12.2
- new net Internal_Tank_Level_Red+: R13.2
- new net Water_Outlet_Valve+: D6.1 (K), Q4.1 (D)
- new net Water_Outlet_Valve-: D6.2 (A), R53.1, R55.2
Other:
- note added: "10"
- note added: "11"
- note added: "12"
- note added: "13"
- note added: "14"
- note added: "15"
- note added: "16"
- note added: "17"
- note added: "18"
- note added: "19"
- note added: "20"
- note added: "21"
- note added: "22"
- note added: "23"
- note added: "24"
- note added: "25"
- note added: "26"
- note added: "27"
- note added: "28"
- note added: "9"
- note added: "IC1 HIGHWAY-C225F 231215Z"
- note added: "U1 VJPN4"
- moved on the sheet: C1, C10, C11, C27, C3, C4, C6, D4, D5, EC1, K2, R15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

Commit message: Update Schematics
Connections:
- net GND: now also C23.1, C24.1
- net IC1_Pin6: no longer C11.1, C6.2
- net at C23.2: now also R49.1
- net Display_RX: now reaches R49.2
- net Water_Tank_Empty+: now reaches R4.1
- net IC1_Pin25: now reaches R4.2
- net TDS+: now reaches R24.1
- net Heater_900W: now reaches R44.1
- net at R50.1: now also C24.2
- net Display_TX: now reaches R50.2
- net UNUSED_CN7+: now reaches C26.2
- net Temperature_Outlet-: now reaches R65.1
- net Relay_Heater_1200W (IC1_Pin2) renamed Heater_1200W
- net U3 Vin renamed U3_Pin1
- new net IC1_Pin13: C11.1, C6.2
Other:
- moved on the sheet: R12, R13

Commit message: Update Schematics
Parts:
- removed C23, C24, C26: unkown, symbol Device:C
- removed D7: D, symbol Device:D
- removed R24, R4, R65: 2kΩ, symbol Device:R
- removed R44: 330Ω, symbol Device:R
- removed R49, R50: 220Ω, symbol Device:R
- added D5: D, symbol Device:D
- added R39: 10kΩ, symbol Device:R
- renumbered D5 to D7
Connections:
- net GND: now also C21.1, Q5.3 (E)
- net Water_Pump+: now also D5.1 (K); no longer D7.1 (K)
- net Water_Pump-: now also D5.2 (A); no longer D7.2 (A)
- net at Q5.1 (C): now also D7.2 (A), K2.A2
- net at Q5.2 (B): now also R39.2
- net at K2.A1: now also C21.2, D7.1 (K)
- net at R34.1: now also R39.1
- net K2_Water_Pump: now reaches R34.2
- net Heater_1200W renamed Heat_1200W
Other:
- added sheet Connectors (MainPCB.Connectors.kicad_sch)
- added sheet MCU (MainPCB.MCU.kicad_sch)
- note removed: "10"
- note removed: "11"
- note removed: "12"
- note removed: "13"
- note removed: "14"
- note removed: "15"
- note removed: "16"
- note removed: "17"
- note removed: "18"
- note removed: "19"
- note removed: "20"
- note removed: "21"
- note removed: "22"
- note removed: "23"
- note removed: "24"
- note removed: "25"
- note removed: "26"
- note removed: "27"
- note removed: "28"
- note removed: "9"
- note removed: "IC1 HIGHWAY-C225F 231215Z"
- moved on the sheet: C10, C11, C12, C13, C14, C15, C16, C17, C2, C20, C22, C25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

Commit message: Update Schematics
Parts:
- removed C14, C17, C2: unkown, symbol Device:C
- removed R12, R13: 2kΩ, symbol Device:R
- RL1: value Ω -> (none)
Connections:
- net GND: now also C11.2, C22.1, C3.2, C4.1, C6.1, Q8.3 (E), R29.1, R40.2, R6.2
- net Heat_1200W: now also R17.2; no longer R17.1
- net IC1_Pin12: now also C11.1, R22.2; no longer C11.2, R22.1
- net K2_Water_Pump: now also R34.1; no longer R34.2
- net U3_Pin1: now also R30.2; no longer R30.1
- net Water_Pump-: no longer R36.2, R64.1
- net at C27.2, R41.1: now also R40.1; no longer R40.2
- net at Q2.3 (S), R15.1: now also R17.1; no longer R17.2
- net at R39.1: now also R34.2; no longer R34.1
- net +5Vdc: now reaches RL1.1
- net +5Vdc: now also C22.2, EC2.1, L1.2
- net IC1_Pin13 renamed IC1_Pin16
- net IC1_Pin16: now also R64.2; no longer C11.1
- removed net Q8_Emitter: C6.1, Q8.3 (E), R64.2
- removed net Transformer+: C10.2, R22.2, R25.1, R30.2, R45.1
- net Transformer- renamed AC_Sense+
- net AC_Sense+: no longer R29.2
- new net: R22.1, R45.1
- new net: R36.2, R64.1
- new net AC_Sense-: C10.2, R25.1, R29.2, R30.1
Other:
- moved on the sheet: C12, C13, C15, C16, C20, C21, C25, C5, C7, C8, C9, D5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
