File: KiCAD/OsmoFresh_Quella_PRO/mainpcb.secondary.kicad_sch (KiCad schematic)
At the start: 79 parts, among them K2 5A 250Vac, Q2 NMOS, Q3 NPN, Q4 PMOS, Q5 NPN, Q6 NPN, Q8 NPN, U4 ULN2003A

Commit message: Update Schematics
Parts:
- added U1: LMV393, symbol Comparator:LMV393
Connections:
- net AC_Sense+: now also R22.1, R45.1
- net GND: now also U1.4 (V-)
- net IC1_Pin11: now also U1.1
- net IC1_Pin3: now also R32.2; no longer R32.1
- net U3_Pin1: now also U1.8 (V+)
- net at Q4.2 (G), R52.2: now also R51.2; no longer R51.1
- net at C27.2, R40.1, R41.1: now also U1.2 (-)
- net at C3.1, R45.2: now also U1.3 (+)
- net at R33.2: now also R32.1; no longer Q8.2 (B)
- net at R33.1: now also Q8.2 (B); no longer R32.2
- net +24Vdc renamed +24V
- net +24V: now also R51.1; no longer R51.2
- net +5Vdc renamed +5V

Commit message: Update Schematics
Parts:
- removed U1: LMV393, symbol Comparator:LMV393
- added U5: KM393, symbol LostCacher:KM393
Connections:
- net U3_Pin1 is gone; now on net +5V: R30.2, R41.2
- net +5V: now also U5.8
- net GND: now also U5.4
- net IC1_Pin11: now also U5.1
- net at C27.2, R40.1, R41.1: now also U5.2
- net at C3.1, R45.2: now also U5.3
Other:
- note removed: "1"
- note removed: "2"
- note removed: "3"
- note removed: "4"
- note removed: "5"
- note removed: "6"
- note removed: "7"
- note removed: "8"
- note removed: "U5 KM393"
- moved on the sheet: C11, C27, R22, R29

Commit message: Update Schematics
Parts:
- removed C1: (no value), symbol Device:C
- removed C10, C12, C13, C15, C16, C18, C19, C20, C21, C22, C25, C27, C4, C5, C7, C8, C9: unkown, symbol Device:C
- removed C11, C3, C6: C, symbol Device:C
- removed D4: (no value), symbol Device:D
- removed D5, D6, D7: D, symbol Device:D
- removed EC1: 470µF 50V, symbol Device:C_Polarized
- removed EC2: 30µF 10V, symbol Device:C_Polarized
- removed K2: 5A 250Vac, symbol Relay:Relay_SPST-NO
- removed L1: (no value), symbol Device:L
- removed Q2: NMOS, symbol Simulation_SPICE:NMOS
- removed Q3, Q5, Q6, Q8: NPN, symbol Simulation_SPICE:NPN
- removed Q4: PMOS, symbol Simulation_SPICE:PMOS
- removed R10, R17, R22, R45, R5, R64, R66: 2kΩ, symbol Device:R
- removed R11, R15, R20, R29, R30, R33, R39, R40, R41, R53, R54, R6, R60, R67, R68: 10kΩ, symbol Device:R
- removed R14, R16, R21, R25: 1kΩ, symbol Device:R
- removed R18, R31: 4,7kΩ, symbol Device:R
- removed R19, R59: 470Ω, symbol Device:R
- removed R23, R61: 47kΩ, symbol Device:R
- removed R32: 5,1kΩ, symbol Device:R
- removed R34: 510Ω, symbol Device:R
- removed R35, R36, R37: 20kΩ, symbol Device:R
- removed R51, R52: 750Ω, symbol Device:R
- removed R55: 5,1Ω, symbol Device:R
- removed R62, R63: 0,62Ω, symbol Device:R
- removed RL1: (no value), symbol Device:R
- removed U4: ULN2003A, symbol Transistor_Array:ULN2003A
- removed U5: KM393, symbol LostCacher:KM393
Other:
- added sheet +24Vdc (MainPCB.+24Vdc.kicad_sch)
- added sheet +5Vdc (MainPCB.5Vdc.kicad_sch)
- note removed: "U1 VJPN4"
- note removed: "Vuanze Electric Y32F-SS-124DM"

Commit message: Update Schematics
Other:
- removed sheet Connectors
Changed lines of the file:
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@@
-		)
-	)
-	(sheet
-		(at 38.1 152.4)
-		(size 38.1 25.4)
-		(exclude_from_sim no)
-		(in_bom yes)
-		(on_board yes)
-		(dnp no)
-		(fields_autoplaced yes)
-		(stroke
-			(width 0.1524)
-			(type solid)
-		)
-		(fill
-			(color 0 0 0 0)
-		)
-		(property "Sheetname" "Connectors"
-			(at 38.1 151.6884 0)
-			(show_name no)
-			(do_not_autoplace no)
-			(effects
-				(font
-					(size 1.27 1.27)
-				)
-				(justify left bottom)
-			)
-		)
-		(property "Sheetfile" "MainPCB.Connectors.kicad_sch"
-			(at 38.1 178.3846 0)
-			(show_name no)
-			(do_not_autoplace no)
-			(effects
-				(font
-					(size 1.27 1.27)
-				)
-				(justify left top)
-			)
-		)
-		(instances
-			(project "OsmoFresh_Quella_PRO"
-				(path "/085f93a2-5d2b-46a2-ac0d-b864eaf3f9e9"
-					(page "6")
-				)
-			)
 		)
 	)

Commit message: Update Schematics
Other:
- sheet +24Vdc: file MainPCB.+24Vdc.kicad_sch -> MainPCB.24Vdc.kicad_sch
Changed lines of the file:
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@@
-	)
-	(sheet
-		(at 38.1 114.3)
-		(size 38.1 25.4)
-		(exclude_from_sim no)
-		(in_bom yes)
-		(on_board yes)
-		(dnp no)
-		(fields_autoplaced yes)
-		(stroke
-			(width 0.1524)
-			(type solid)
-		)
-		(fill
-			(color 0 0 0 0)
-		)
-		(property "Sheetname" "MCU"
-			(at 38.1 113.5884 0)
-			(show_name no)
-			(do_not_autoplace no)
-			(effects
-				(font
-					(size 1.27 1.27)
-				)
-				(justify left bottom)
-			)
-		)
-		(property "Sheetfile" "MainPCB.MCU.kicad_sch"
-			(at 38.1 140.2846 0)
-			(show_name no)
-			(do_not_autoplace no)
-			(effects
-				(font
-					(size 1.27 1.27)
-				)
-				(justify left top)
-			)
-		)
-		(instances
-			(project "OsmoFresh_Quella_PRO"
-				(path "/085f93a2-5d2b-46a2-ac0d-b864eaf3f9e9"
-					(page "5")
-				)
-			)
-		)
-	)
-	(sheet
-		(at 38.1 77.47)
-		(size 38.1 25.4)
-		(exclude_from_sim no)
-		(in_bom yes)
-		(on_board yes)
-		(dnp no)
-		(fields_autoplaced yes)
-		(stroke
-			(width 0.1524)
-			(type solid)
-		)
-		(fill
-			(color 0 0 0 0)
-		)
-		(property "Sheetname" "+5Vdc"
-			(at 38.1 76.7584 0)
-			(show_name no)
-			(do_not_autoplace no)
-			(effects
-				(font
-					(size 1.27 1.27)
-				)
-				(justify left bottom)
-			)
-		)
-		(property "Sheetfile" "MainPCB.5Vdc.kicad_sch"
-			(at 38.1 103.4546 0)
-			(show_name no)
-			(do_not_autoplace no)
-			(effects
-				(font
-					(size 1.27 1.27)
-				)
-				(justify left top)
-			)
-		)
-		(instances
-			(project "OsmoFresh_Quella_PRO"
-				(path "/085f93a2-5d2b-46a2-ac0d-b864eaf3f9e9"
-					(page "4")
-				)
-			)
-		)
 	)
 	(sheet
@@
 			)
 		)
-		(property "Sheetfile" "MainPCB.+24Vdc.kicad_sch"
+		(property "Sheetfile" "MainPCB.24Vdc.kicad_sch"
 			(at 38.1 64.0846 0)
 			(show_name no)
@@
 		(instances
 			(project "OsmoFresh_Quella_PRO"
-				(path "/085f93a2-5d2b-46a2-ac0d-b864eaf3f9e9"
+				(path "/4260df0e-d900-46a1-97d3-cde6b2933985"
 					(page "3")
 				)
 			)
+		)
+	)
+	(sheet
+		(at 139.7 38.1)
+		(size 38.1 25.4)
+		(exclude_from_sim no)
+		(in_bom yes)
+		(on_board yes)
+		(dnp no)
+		(fields_autoplaced yes)
+		(stroke
+			(width 0.1524)
+			(type solid)
+		)
+		(fill
+			(color 0 0 0 0)
+		)
+		(property "Sheetname" "MCU"
+			(at 139.7 37.3884 0)
+			(show_name no)
+			(do_not_autoplace no)
+			(effects
+				(font
+					(size 1.27 1.27)
+				)
+				(justify left bottom)
+			)
+		)
+		(property "Sheetfile" "MainPCB.MCU.kicad_sch"
+			(at 139.7 64.0846 0)
+			(show_name no)
+			(do_not_autoplace no)
+			(effects
+				(font
+					(size 1.27 1.27)
+				)
+				(justify left top)
+			)
+		)
+		(instances
+			(project "OsmoFresh_Quella_PRO"
+				(path "/4260df0e-d900-46a1-97d3-cde6b2933985"
+					(page "5")
+				)
+			)
+		)
+	)
+	(sheet
+		(at 88.9 38.1)
+		(size 38.1 25.4)
+		(exclude_from_sim no)
+		(in_bom yes)
+		(on_board yes)
+		(dnp no)
+		(fields_autoplaced yes)
+		(stroke
+			(width 0.1524)
+			(type solid)
+		)
+		(fill
+			(color 0 0 0 0)
+		)
+		(property "Sheetname" "+5Vdc"
+			(at 88.9 37.3884 0)
+			(show_name no)
+			(do_not_autoplace no)
+			(effects
+				(font
+					(size 1.27 1.27)
+				)
+				(justify left bottom)
+			)
+		)
+		(property "Sheetfile" "MainPCB.5Vdc.kicad_sch"
+			(at 88.9 64.0846 0)
+			(show_name no)
+			(do_not_autoplace no)
+			(effects
+				(font
+					(size 1.27 1.27)
+				)
+				(justify left top)
+			)
+		)
+		(instances
+			(project "OsmoFresh_Quella_PRO"
+				(path "/4260df0e-d900-46a1-97d3-cde6b2933985"
+					(page "4")
+				)
+			)

Commit message: Update Schematics
Changed lines of the file:
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@@
 	(title_block
 		(title "MainPCB Secondary")
-		(date "2026-08-15")
+		(date "2026-08-20")
 		(rev "1.0.0")
 		(company "LostCacher")
 	)
 	(sheet
-		(at 38.1 38.1)
-		(size 38.1 25.4)
+		(at 25.4 63.5)
+		(size 63.5 63.5)
 		(exclude_from_sim no)
 		(in_bom yes)
@@
 		)
 		(property "Sheetname" "+24Vdc"
-			(at 38.1 37.3884 0)
+			(at 25.4 62.7884 0)
 			(show_name no)
 			(do_not_autoplace no)
@@
 		)
 		(property "Sheetfile" "MainPCB.24Vdc.kicad_sch"
-			(at 38.1 64.0846 0)
+			(at 25.4 127.5846 0)
 			(show_name no)
 			(do_not_autoplace no)
@@
 	)
 	(sheet
-		(at 139.7 38.1)
-		(size 38.1 25.4)
+		(at 203.2 63.5)
+		(size 63.5 63.5)
 		(exclude_from_sim no)
 		(in_bom yes)
@@
 		)
 		(property "Sheetname" "MCU"
-			(at 139.7 37.3884 0)
+			(at 203.2 62.7884 0)
 			(show_name no)
 			(do_not_autoplace no)
@@
 		)
 		(property "Sheetfile" "MainPCB.MCU.kicad_sch"
-			(at 139.7 64.0846 0)
+			(at 203.2 127.5846 0)
 			(show_name no)
 			(do_not_autoplace no)
@@
 	)
 	(sheet
-		(at 88.9 38.1)
-		(size 38.1 25.4)
+		(at 114.3 63.5)
+		(size 63.5 63.5)
 		(exclude_from_sim no)
 		(in_bom yes)
@@
 		)
 		(property "Sheetname" "+5Vdc"
-			(at 88.9 37.3884 0)
+			(at 114.3 62.7884 0)
 			(show_name no)
 			(do_not_autoplace no)
@@
 		)
 		(property "Sheetfile" "MainPCB.5Vdc.kicad_sch"
-			(at 88.9 64.0846 0)
+			(at 114.3 127.5846 0)
 			(show_name no)
 			(do_not_autoplace no)
