File: KiCAD/OsmoFresh_Quella_PRO/MainPCB.Connectors.kicad_sch (KiCad schematic)
At the start: 14 parts, among them CN15 Conn_01x04_Pin, CN17 Conn_01x02_Pin, CN18 Conn_01x02_Pin, CN19 Conn_01x02_Pin, CN20 Conn_01x02_Pin, CN21 Conn_01x02_Pin, CN22 Conn_01x02_Pin, CN23 Conn_01x02_Pin, CN24 Conn_01x02_Pin, CN25 Conn_01x02_Pin, CN26 Conn_01x02_Pin, CN27 Conn_01x06_Pin, CN28 Conn_01x02_Pin, CN4 Conn_01x02_Pin

Commit message: Update Schematics
Parts:
- renumbered CN28 to CN1, CN27 to CN10, CN15 to CN11, CN25 to CN12, CN26 to CN13, CN23 to CN14, CN18 to CN16, CN22 to CN2, CN4 to CN3, CN17 to CN5, CN24 to CN6, CN21 to CN7, CN19 to CN8, CN20 to CN9
Connections:
- net +24Vdc renamed +24V
- net +5Vdc renamed +5V
Other:
- moved on the sheet: CN11, CN12, CN13, CN14, CN16, CN2, CN3, CN5, CN6, CN7, CN8, CN9

Commit message: Update Schematics
Other:
- title: MainPCB Secondary Connectors -> MainPCB Connectors
Changed lines of the file:
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@@
 	(paper "A4")
 	(title_block
-		(title "MainPCB Secondary Connectors")
-		(date "2026-08-14")
+		(title "MainPCB Connectors")
+		(date "2026-08-15")
 		(rev "1.0.0")
 		(company "LostCacher")
