File: KiCAD/OsmoFresh_Quella_PRO/OsmoFresh_Quella_PRO.kicad_sch (KiCad schematic)
At the start: 11 parts, among them K1 10A 250Vac, Q1 BTA16-800CW, SW1 [NC]

Commit message: Update Schematics
Parts:
- R26, R27, R28: value 82 kΩ -> 82kΩ
- R7: value 180 Ω -> 180Ω
Connections:
- net CURRENT_SENSE+ renamed Current_Sense+
- net CURRENT_SENSE- renamed Current_Sense-
- net RELAY_HEATER_COIL+ renamed Relay_Heater_Coil+
- net RELAY_HEATER_COIL- renamed Relay_Heater_Colil-
Other:
- title: MainPCB.Primary -> MainPCB Primary
Changed lines of the file:
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@@
 	(paper "A4")
 	(title_block
-		(title "MainPCB.Primary")
+		(title "MainPCB Primary")
 		(date "2026-08-12")
 		(rev "1.0.0")
@@
 		)
 	)
-	(global_label "RELAY_HEATER_COIL+"
+	(global_label "Relay_Heater_Coil+"
 		(shape input)
 		(at 147.32 63.5 0)
@@
 		)
 		(property "Intersheetrefs" "${INTERSHEET_REFS}"
-			(at 170.6252 63.5 0)
+			(at 168.8108 63.5 0)
 			(hide yes)
 			(show_name no)
@@
 		)
 	)
-	(global_label "TEMP_OUT+"
+	(global_label "Temp_Out+"
 		(shape output)
 		(at 236.22 46.99 180)
@@
 		)
 		(property "Intersheetrefs" "${INTERSHEET_REFS}"
-			(at 222.2282 46.99 0)
+			(at 222.5911 46.99 0)
 			(hide yes)
 			(show_name no)
@@
 		)
 	)
-	(global_label "CURRENT_SENSE-"
+	(global_label "Current_Sense-"
 		(shape output)
 		(at 62.23 49.53 90)
@@
 		)
 		(property "Intersheetrefs" "${INTERSHEET_REFS}"
-			(at 62.23 29.3697 90)
+			(at 62.23 31.4863 90)
 			(hide yes)
 			(show_name no)
@@
 		)
 	)
-	(global_label "TEMP_OUT-"
+	(global_label "Temp_Out-"
 		(shape output)
 		(at 236.22 50.8 180)
@@
 		)
 		(property "Intersheetrefs" "${INTERSHEET_REFS}"
-			(at 222.2282 50.8 0)
+			(at 222.5911 50.8 0)
 			(hide yes)
 			(show_name no)
@@
 		)
 	)
-	(global_label "CURRENT_SENSE+"
+	(global_label "Current_Sense+"
 		(shape output)
 		(at 72.39 49.53 90)
@@
 		)
 		(property "Intersheetrefs" "${INTERSHEET_REFS}"
-			(at 72.39 29.3697 90)
+			(at 72.39 31.4863 90)
 			(hide yes)
 			(show_name no)
@@
 		)
 	)
-	(global_label "RELAY_HEATER_COIL-"
+	(global_label "Relay_Heater_Colil-"
 		(shape input)
 		(at 127 63.5 180)
@@
 		)
 		(property "Intersheetrefs" "${INTERSHEET_REFS}"
-			(at 103.6948 63.5 0)
+			(at 104.844 63.5 0)
 			(hide yes)
 			(show_name no)
@@
 			)
 		)
-		(property "Value" "82 kΩ"
+		(property "Value" "82kΩ"
 			(at 60.96 109.2199 0)
 			(show_name no)
@@
 			)
 		)
-		(property "Value" "180 Ω"
+		(property "Value" "180Ω"
 			(at 90.17 114.3 90)
 			(show_name no)
@@
 			)
 		)
-		(property "Value" "82 kΩ"
+		(property "Value" "82kΩ"
 			(at 60.96 86.3599 0)
 			(show_name no)
@@
 			)
 		)
-		(property "Value" "82 kΩ"
+		(property "Value" "82kΩ"
 			(at 60.96 97.7899 0)
 			(show_name no)

Commit message: Update Schematics
Connections:
- net Current_Sense+ renamed Transformer+
- net Current_Sense- renamed Transformer-
Changed lines of the file:
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@@
+	(wire
+		(pts
+			(xy 151.13 118.11) (xy 142.24 118.11)
+		)
+		(stroke
+			(width 0)
+			(type default)
+		)
+	)
 	(wire
 		(pts
@@
 	(wire
 		(pts
+			(xy 93.98 116.84) (xy 110.49 116.84)
+		)
+		(stroke
+			(width 0)
+			(type default)
+		)
+	)
+	(wire
+		(pts
 			(xy 77.47 92.71) (xy 77.47 116.84)
 		)
@@
 	(wire
 		(pts
+			(xy 142.24 118.11) (xy 142.24 119.38)
+		)
+		(stroke
+			(width 0)
+			(type default)
+		)
+	)
+	(wire
+		(pts
 			(xy 121.92 100.33) (xy 121.92 105.41)
 		)
@@
 		(pts
 			(xy 243.84 107.95) (xy 243.84 105.41)
-		)
-		(stroke
-			(width 0)
-			(type default)
-		)
-	)
-	(wire
-		(pts
-			(xy 93.98 116.84) (xy 110.49 116.84)
 		)
 		(stroke
@@
 		)
 	)
-	(global_label "Current_Sense-"
+	(global_label "Transformer-"
 		(shape output)
 		(at 62.23 49.53 90)
@@
 		)
 		(property "Intersheetrefs" "${INTERSHEET_REFS}"
-			(at 62.23 31.4863 90)
+			(at 62.23 33.6635 90)
 			(hide yes)
 			(show_name no)
@@
 		)
 	)
+	(global_label "U3 Vin"
+		(shape input)
+		(at 151.13 118.11 0)
+		(fields_autoplaced yes)
+		(effects
+			(font
+				(size 1.27 1.27)
+			)
+			(justify left)
+		)
+		(property "Intersheetrefs" "${INTERSHEET_REFS}"
+			(at 160.4652 118.11 0)
+			(hide yes)
+			(show_name no)
+			(do_not_autoplace no)
+			(effects
+				(font
+					(size 1.27 1.27)
+				)
+				(justify left)
+			)
+		)
+	)
 	(global_label "Heater_Neutral"
 		(shape output)
@@
 		)
 	)
-	(global_label "Current_Sense+"
+	(global_label "Transformer+"
 		(shape output)
 		(at 72.39 49.53 90)
@@
 		)
 		(property "Intersheetrefs" "${INTERSHEET_REFS}"
-			(at 72.39 31.4863 90)
-			(hide yes)
-			(show_name no)
+			(at 72.39 33.6635 90)
+			(hide yes)
+			(show_name no)

Commit message: Update Schematics
Changed lines of the file:
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@@
+	(wire
+		(pts
+			(xy 137.16 111.76) (xy 137.16 119.38)
+		)
+		(stroke
+			(width 0)
+			(type default)
+		)
+	)
 	(wire
 		(pts
@@
 		(pts
 			(xy 110.49 124.46) (xy 124.46 124.46)
+		)
+		(stroke
+			(width 0)
+			(type default)
+		)
+	)
+	(wire
+		(pts
+			(xy 151.13 111.76) (xy 137.16 111.76)
 		)
 		(stroke
@@
 		)
 	)
+	(global_label "Heater_900W"
+		(shape input)
+		(at 151.13 111.76 0)
+		(fields_autoplaced yes)
+		(effects
+			(font
+				(size 1.27 1.27)
+			)
+			(justify left)
+		)
+		(property "Intersheetrefs" "${INTERSHEET_REFS}"
+			(at 166.3313 111.76 0)
+			(hide yes)
+			(show_name no)
+			(do_not_autoplace no)
+			(effects
+				(font
+					(size 1.27 1.27)
+				)
+				(justify left)
+			)
+		)
+	)
 	(global_label "Temp_Out+"
 		(shape output)
@@
 		)
 	)
-	(global_label "U3 Vin"
+	(global_label "U3_Pin1"
 		(shape input)
 		(at 151.13 118.11 0)
@@
 		)
 		(property "Intersheetrefs" "${INTERSHEET_REFS}"
-			(at 160.4652 118.11 0)
-			(hide yes)
-			(show_name no)
+			(at 161.8561 118.11 0)
+			(hide yes)
+			(show_name no)

Commit message: Update Schematics
Changed lines of the file:
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@@
 	(title_block
 		(title "MainPCB Primary")
-		(date "2026-08-12")
+		(date "2026-08-13")
 		(rev "1.0.0")
 		(company "LostCacher")
@@
 	(text "Vuanze Electric Y32F-SS-124HM"
 		(exclude_from_sim no)
-		(at 137.414 56.642 0)
+		(at 136.652 81.534 0)
 		(effects
 			(font
@@
 		)
 	)
-	(global_label "Heater_900W"
+	(global_label "Heat_900W"
 		(shape input)
 		(at 151.13 111.76 0)
@@
 		)
 		(property "Intersheetrefs" "${INTERSHEET_REFS}"
-			(at 166.3313 111.76 0)
+			(at 164.4565 111.76 0)
 			(hide yes)
 			(show_name no)
@@
 		(dnp no)
 		(property "Reference" "K1"
-			(at 137.16 51.308 90)
+			(at 137.16 54.356 90)
 			(show_name no)
 			(do_not_autoplace no)
@@
 		)
 		(property "Value" "10A 250Vac"
-			(at 137.16 53.848 90)
-			(show_name no)
-			(do_not_autoplace no)
+			(at 137.16 56.896 90)
+			(show_name no)
+			(do_not_autoplace no)

Commit message: Update Schematics
Connections:
- net Transformer+ renamed AC_Sense+
- net Transformer- renamed AC_Sense-
Changed lines of the file:
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@@
 		)
 	)
-	(global_label "Transformer-"
+	(global_label "AC_Sense-"
 		(shape output)
 		(at 62.23 49.53 90)
@@
 		)
 		(property "Intersheetrefs" "${INTERSHEET_REFS}"
-			(at 62.23 33.6635 90)
+			(at 62.23 36.0824 90)
 			(hide yes)
 			(show_name no)
@@
 		)
 	)
-	(global_label "Transformer+"
+	(global_label "AC_Sense+"
 		(shape output)
 		(at 72.39 49.53 90)
@@
 		)
 		(property "Intersheetrefs" "${INTERSHEET_REFS}"
-			(at 72.39 33.6635 90)
+			(at 72.39 36.0824 90)
 			(hide yes)
 			(show_name no)

Commit message: Update Schematics
Parts:
- added P3, P4, P5, P6, P7: (no value), symbol My_Default:Faston_6.3mm_1Pin
Connections:
- net Heater_Neutral: now also P3., P4., P7.
- net at FUSE1.1, K1.13, Q1.2 (A2)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: now also P5.
- net at FUSE1.2: now also P6.
Other:
- note removed: "P10"
- note removed: "P3"
- note removed: "P4"
- note removed: "P5"
- note removed: "P6"

Commit message: Update Schematics
Changed lines of the file:
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@@
 		)
 	)
-	(global_label "U3_Pin1"
-		(shape input)
-		(at 151.13 118.11 0)
+	(global_label "Heater_Neutral"
+		(shape output)
+		(at 41.91 139.7 180)
 		(fields_autoplaced yes)
 		(effects
@@
 				(size 1.27 1.27)
 			)
-			(justify left)
+			(justify right)
 		)
 		(property "Intersheetrefs" "${INTERSHEET_REFS}"
-			(at 161.8561 118.11 0)
-			(hide yes)
-			(show_name no)
-			(do_not_autoplace no)
-			(effects
-				(font
-					(size 1.27 1.27)
-				)
-				(justify left)
-			)
-		)
-	)
-	(global_label "Heater_Neutral"
+			(at 24.8944 139.7 0)
+			(hide yes)
+			(show_name no)
+			(do_not_autoplace no)
+			(effects
+				(font
+					(size 1.27 1.27)
+				)
+				(justify right)
+			)
+		)
+	)
+	(global_label "Temp_Out-"
 		(shape output)
-		(at 41.91 139.7 180)
+		(at 236.22 50.8 180)
 		(fields_autoplaced yes)
 		(effects
@@
 		)
 		(property "Intersheetrefs" "${INTERSHEET_REFS}"
-			(at 24.8944 139.7 0)
+			(at 222.5911 50.8 0)
 			(hide yes)
 			(show_name no)
@@
 		)
 	)
-	(global_label "Temp_Out-"
+	(global_label "Heater_900W"
 		(shape output)
-		(at 236.22 50.8 180)
+		(at 125.73 105.41 0)
 		(fields_autoplaced yes)
 		(effects
@@
 				(size 1.27 1.27)
 			)
-			(justify right)
+			(justify left)
 		)
 		(property "Intersheetrefs" "${INTERSHEET_REFS}"
-			(at 222.5911 50.8 0)
-			(hide yes)
-			(show_name no)
-			(do_not_autoplace no)
-			(effects
-				(font
-					(size 1.27 1.27)
-				)
-				(justify right)
+			(at 140.9313 105.41 0)
+			(hide yes)
+			(show_name no)
+			(do_not_autoplace no)
+			(effects
+				(font
+					(size 1.27 1.27)
+				)
+				(justify left)
 			)
 		)
 	)
 	(global_label "Heater_900W"
-		(shape output)
-		(at 125.73 105.41 0)
+		(shape input)
+		(at 236.22 88.9 180)
 		(fields_autoplaced yes)
 		(effects
@@
 				(size 1.27 1.27)
 			)
-			(justify left)
+			(justify right)
 		)
 		(property "Intersheetrefs" "${INTERSHEET_REFS}"
-			(at 140.9313 105.41 0)
-			(hide yes)
-			(show_name no)
-			(do_not_autoplace no)
-			(effects
-				(font
-					(size 1.27 1.27)
-				)
-				(justify left)
-			)
-		)
-	)
-	(global_label "Heater_900W"
-		(shape input)
-		(at 236.22 88.9 180)
+			(at 221.0187 88.9 0)
+			(hide yes)
+			(show_name no)
+			(do_not_autoplace no)
+			(effects
+				(font
+					(size 1.27 1.27)
+				)
+				(justify right)
+			)
+		)
+	)
+	(global_label "AC_Sense+"
+		(shape output)
+		(at 72.39 49.53 90)
 		(fields_autoplaced yes)
 		(effects
@@
 				(size 1.27 1.27)
 			)
-			(justify right)
+			(justify left)
 		)
 		(property "Intersheetrefs" "${INTERSHEET_REFS}"
-			(at 221.0187 88.9 0)
-			(hide yes)
-			(show_name no)
-			(do_not_autoplace no)
-			(effects
-				(font
-					(size 1.27 1.27)
-				)
-				(justify right)
-			)
-		)
-	)
-	(global_label "AC_Sense+"
-		(shape output)
-		(at 72.39 49.53 90)
+			(at 72.39 36.0824 90)
+			(hide yes)
+			(show_name no)
+			(do_not_autoplace no)
+			(effects
+				(font
+					(size 1.27 1.27)
+				)
+				(justify left)
+			)
+		)
+	)
+	(global_label "Relay_Heater_Colil-"
+		(shape input)
+		(at 127 63.5 180)
 		(fields_autoplaced yes)
 		(effects
@@
 				(size 1.27 1.27)
 			)
-			(justify left)
-		)
-		(property "Intersheetrefs" "${INTERSHEET_REFS}"
-			(at 72.39 36.0824 90)
-			(hide yes)
-			(show_name no)
-			(do_not_autoplace no)
-			(effects
-				(font
-					(size 1.27 1.27)
-				)
-				(justify left)
-			)
-		)
-	)
-	(global_label "Relay_Heater_Colil-"
-		(shape input)
-		(at 127 63.5 180)
-		(fields_autoplaced yes)
-		(effects
-			(font
-				(size 1.27 1.27)
-			)
 			(justify right)
 		)
@@
 					(unit 1)
 				)
+			)
+		)
+	)
+	(symbol
+		(lib_id "power:+5V")
+		(at 151.13 118.11 270)
+		(unit 1)
+		(body_style 1)
+		(exclude_from_sim no)
+		(in_bom yes)
+		(on_board yes)
+		(in_pos_files yes)
+		(dnp no)
+		(fields_autoplaced yes)
+		(property "Reference" "#PWR07"
+			(at 147.32 118.11 0)
+			(hide yes)
+			(show_name no)
+			(do_not_autoplace no)
+			(effects
+				(font
+					(size 1.27 1.27)
+				)
+			)
+		)
+		(property "Value" "+5V"
+			(at 154.94 118.1099 90)
+			(show_name no)
+			(do_not_autoplace no)
+			(effects
+				(font
+					(size 1.27 1.27)
+				)
+				(justify left)
+			)
+		)
+		(property "Footprint" ""
+			(at 151.13 118.11 0)
+			(hide yes)
+			(show_name no)
+			(do_not_autoplace no)
+			(effects
+				(font
+					(size 1.27 1.27)
+				)
+			)
+		)
+		(property "Datasheet" ""
+			(at 151.13 118.11 0)
+			(hide yes)
+			(show_name no)
+			(do_not_autoplace no)
+			(effects
+				(font
+					(size 1.27 1.27)
+				)
+			)
+		)
+		(property "Description" "Power symbol creates a global label with name \"+5V\""
+			(at 151.13 118.11 0)
+			(hide yes)
+			(show_name no)
+			(do_not_autoplace no)
+			(effects
+				(font
+					(size 1.27 1.27)
+				)
+			)
+		)
+		(pin "1"
+		)
+		(instances
+			(project "OsmoFresh_Quella_PRO"
+				(path "/fa934e2d-e6dc-4af7-b9d3-1332cdb541a5"
+					(reference "#PWR07")
+					(unit 1)
+				)
