File: KiCAD/OsmoFresh_Quella_PRO/OsmoFresh_Quella_PRO.kicad_sch (KiCad schematic)
At the start: 16 parts, among them K1 10A 250Vac, Q1 BTA16-800CW, SW1 [NC]

Commit message: Update Schematics
Parts:
- added R46: 330Ω, symbol Device:R
Connections:
- net Heat_900W: now also R46.1
Changed lines of the file:
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@@
+	(wire
+		(pts
+			(xy 137.16 111.76) (xy 140.97 111.76)
+		)
+		(stroke
+			(width 0)
+			(type default)
+		)
+	)
 	(wire
 		(pts
@@
 	(wire
 		(pts
-			(xy 151.13 111.76) (xy 137.16 111.76)
-		)
-		(stroke
-			(width 0)
-			(type default)
-		)
-	)
-	(wire
-		(pts
 			(xy 113.03 99.06) (xy 113.03 121.92)
 		)
@@
 		(pts
 			(xy 142.24 139.7) (xy 142.24 147.32)
+		)
+		(stroke
+			(width 0)
+			(type default)
+		)
+	)
+	(wire
+		(pts
+			(xy 148.59 111.76) (xy 152.4 111.76)
 		)
 		(stroke
@@
 	(global_label "Heat_900W"
 		(shape input)
-		(at 151.13 111.76 0)
+		(at 152.4 111.76 0)
 		(fields_autoplaced yes)
 		(effects
@@
 		)
 		(property "Intersheetrefs" "${INTERSHEET_REFS}"
-			(at 164.4565 111.76 0)
+			(at 165.7265 111.76 0)
 			(hide yes)
 			(show_name no)
@@
 		)
 	)
-	(global_label "Temp_Out+"
+	(global_label "Temperature_Outlet+"
 		(shape output)
 		(at 236.22 46.99 180)
@@
 		)
 		(property "Intersheetrefs" "${INTERSHEET_REFS}"
-			(at 222.5911 46.99 0)
+			(at 213.3383 46.99 0)
 			(hide yes)
 			(show_name no)
@@
 		)
 	)
-	(global_label "Temp_Out-"
+	(global_label "Temperature_Outlet-"
 		(shape output)
 		(at 236.22 50.8 180)
@@
 		)
 		(property "Intersheetrefs" "${INTERSHEET_REFS}"
-			(at 222.5911 50.8 0)
+			(at 213.3383 50.8 0)
 			(hide yes)
 			(show_name no)
@@
 					(unit 1)
 				)
+			)
+		)
+	)
+	(symbol
+		(lib_id "Device:R")
+		(at 144.78 111.76 270)
+		(unit 1)
+		(body_style 1)
+		(exclude_from_sim no)
+		(in_bom yes)
+		(on_board yes)
+		(in_pos_files yes)
+		(dnp no)
+		(property "Reference" "R46"
+			(at 144.78 107.696 90)
+			(show_name no)
+			(do_not_autoplace no)
+			(effects
+				(font
+					(size 1.27 1.27)
+				)
+			)
+		)
+		(property "Value" "330Ω"
+			(at 144.78 109.474 90)
+			(show_name no)
+			(do_not_autoplace no)
+			(effects
+				(font
+					(size 1.27 1.27)
+				)
+			)
+		)
+		(property "Footprint" ""
+			(at 144.78 109.982 90)
+			(hide yes)
+			(show_name no)
+			(do_not_autoplace no)
+			(effects
+				(font
+					(size 1.27 1.27)
+				)
+			)
+		)
+		(property "Datasheet" ""
+			(at 144.78 111.76 0)
+			(hide yes)
+			(show_name no)
+			(do_not_autoplace no)
+			(effects
+				(font
+					(size 1.27 1.27)
+				)
+			)
+		)
+		(property "Description" "Resistor"
+			(at 144.78 111.76 0)
+			(hide yes)
+			(show_name no)
+			(do_not_autoplace no)
+			(effects
+				(font
+					(size 1.27 1.27)
+				)
+			)
+		)
+		(pin "1"
+		)
+		(pin "2"
+		)
+		(instances
+			(project "OsmoFresh_Quella_PRO"
+				(path "/fa934e2d-e6dc-4af7-b9d3-1332cdb541a5"
+					(reference "R46")
+					(unit 1)
+				)

Commit message: Update Schematics
Parts:
- XC1: value 0,1µF -> 100nF
- renumbered R46 to R44
Changed lines of the file:
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@@
 		(in_pos_files yes)
 		(dnp no)
-		(property "Reference" "R46"
+		(property "Reference" "R44"
 			(at 144.78 107.696 90)
 			(show_name no)
@@
 			(project "OsmoFresh_Quella_PRO"
 				(path "/fa934e2d-e6dc-4af7-b9d3-1332cdb541a5"
-					(reference "R46")
+					(reference "R44")
 					(unit 1)
 				)
@@
 			)
 		)
-		(property "Value" "0,1µF"
+		(property "Value" "100nF"
 			(at 68.58 133.604 90)
 			(show_name no)

Commit message: Update Schematics
Parts:
- removed K1: 10A 250Vac, symbol Relay:Relay_SPST-NO
- removed R44: 330Ω, symbol Device:R
- removed R7: 180Ω, symbol Device:R
Connections:
- net LINE: now reaches FUSE1.1, P5., Q1.2 (A2), T1.2 (AB), XC1.2, ZNR1.2
- net Heater_Triac_Gate: now reaches Q1.3 (G)
- net Heater_Neutral renamed NEUT
Other:
- note removed: "1"
- note removed: "2"
- note removed: "3"
- note removed: "4"
- note removed: "5"
- note removed: "6"
- note removed: "U3 UNKNOWN"
- note removed: "Vuanze Electric Y32F-SS-124HM"
- moved on the sheet: FUSE1, P3, P4, P5, P6, P7, Q1, R26, R27, R28, T1, XC1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
