File: KiCAD/OsmoFresh_Quella_PRO/MainPCB.+24Vdc.kicad_sch (KiCad schematic)
At the start: 63 parts, among them K2 5A 250Vac, Q2 NMOS, Q3 NPN, Q4 PMOS, Q5 NPN, Q6 NPN, Q8 NPN, U4 ULN2003A

Commit message: Update Schematics
Parts:
- added CN1, CN12, CN13: Conn_01x02_Pin, symbol Connector:Conn_01x02_Pin
- added CN10: Conn_01x06_Pin, symbol Connector:Conn_01x06_Pin
Connections:
- net +24V: now also CN1.1 (Pin_1), CN10.2 (Pin_2), CN10.4 (Pin_4), CN13.1 (Pin_1)
- net Flush_Valve-: now also CN10.3 (Pin_3)
- net GND: now also CN1.2 (Pin_2)
- net UNUSED_CN10-: now also CN10.1 (Pin_1)
- net UNUSED_CN13-: now also CN13.2 (Pin_2)
- net Water_Outlet_Valve+: now also CN12.1 (Pin_1)
- net Water_Outlet_Valve-: now also CN12.2 (Pin_2)
- net Water_Pump+: now also CN10.6 (Pin_6)
- net Water_Pump-: now also CN10.5 (Pin_5)
