File: KiCAD/OsmoFresh_Quella_PRO/MainPCB.MCU.kicad_sch (KiCad schematic)
At the start: 9 parts

Commit message: Update Schematics
Parts:
- added C14, C17, C2: unkown, symbol Device:C
- added R12, R13: 2kΩ, symbol Device:R
Connections:
- net GND: now also C14.1, C17.1, C2.1
- new net +5Vdc: C14.2, C17.2, C2.2
- new net Internal_Tank_Level_Black+: R12.2
- new net Internal_Tank_Level_Red+: R13.2

Commit message: Update Schematics
Connections:
- net +5Vdc renamed +5V
Changed lines of the file:
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@@
 	(title_block
 		(title "MainPCB MCU")
-		(date "2026-08-13")
+		(date "2026-08-14")
 		(rev "1.0.0")
 		(company "LostCacher")
@@
 	(wire
 		(pts
-			(xy 177.8 50.8) (xy 177.8 55.88)
-		)
-		(stroke
-			(width 0)
-			(type default)
-		)
-	)
-	(wire
-		(pts
 			(xy 144.78 129.54) (xy 140.97 129.54)
 		)
@@
 		)
 	)
-	(global_label "GND"
-		(shape input)
-		(at 228.6 69.85 0)
-		(fields_autoplaced yes)
-		(effects
-			(font
-				(size 1.27 1.27)
-			)
-			(justify left)
-		)
-		(property "Intersheetrefs" "${INTERSHEET_REFS}"
-			(at 235.4557 69.85 0)
-			(hide yes)
-			(show_name no)
-			(do_not_autoplace no)
-			(effects
-				(font
-					(size 1.27 1.27)
-				)
-				(justify left)
-			)
-		)
-	)
 	(global_label "UNUSED_CN7-"
 		(shape output)
@@
 	)
 	(global_label "IC1_Pin12"
-		(shape input)
+		(shape bidirectional)
 		(at 177.8 73.66 0)
 		(fields_autoplaced yes)
@@
 		)
 		(property "Intersheetrefs" "${INTERSHEET_REFS}"
-			(at 190.2799 73.66 0)
+			(at 191.3912 73.66 0)
 			(hide yes)
 			(show_name no)
@@
 	)
 	(global_label "IC1_Pin15"
-		(shape output)
+		(shape input)
 		(at 120.65 66.04 180)
 		(fields_autoplaced yes)
@@
 		)
 	)
-	(global_label "+5Vdc"
-		(shape input)
-		(at 177.8 50.8 90)
-		(fields_autoplaced yes)
-		(effects
-			(font
-				(size 1.27 1.27)
-			)
-			(justify left)
-		)
-		(property "Intersheetrefs" "${INTERSHEET_REFS}"
-			(at 177.8 41.7067 90)
-			(hide yes)
-			(show_name no)
-			(do_not_autoplace no)
-			(effects
-				(font
-					(size 1.27 1.27)
-				)
-				(justify left)
-			)
-		)
-	)
-	(global_label "GND"
-		(shape input)
-		(at 140.97 132.08 270)
-		(fields_autoplaced yes)
-		(effects
-			(font
-				(size 1.27 1.27)
-			)
-			(justify right)
-		)
-		(property "Intersheetrefs" "${INTERSHEET_REFS}"
-			(at 140.97 138.9357 90)
-			(hide yes)
-			(show_name no)
-			(do_not_autoplace no)
-			(effects
-				(font
-					(size 1.27 1.27)
-				)
-				(justify right)
-			)
-		)
-	)
 	(global_label "TDS+"
 		(shape input)
@@
 		)
 	)
-	(global_label "UNUSED_CN16+"
-		(shape bidirectional)
-		(at 92.71 110.49 180)
-		(fields_autoplaced yes)
-		(effects
-			(font
-				(size 1.27 1.27)
-			)
-			(justify right)
-		)
-		(property "Intersheetrefs" "${INTERSHEET_REFS}"
-			(at 73.434 110.49 0)
-			(hide yes)
-			(show_name no)
-			(do_not_autoplace no)
-			(effects
-				(font
-					(size 1.27 1.27)
-				)
-				(justify right)
-			)
-		)
-	)
 	(global_label "Heat_1200W"
 		(shape output)
@@
 		(property "Intersheetrefs" "${INTERSHEET_REFS}"
 			(at 155.644 127 0)
-			(hide yes)
-			(show_name no)
-			(do_not_autoplace no)
-			(effects
-				(font
-					(size 1.27 1.27)
-				)
-				(justify right)
-			)
-		)
-	)
-	(global_label "UNUSED_CN16-"
-		(shape bidirectional)
-		(at 92.71 106.68 180)
-		(fields_autoplaced yes)
-		(effects
-			(font
-				(size 1.27 1.27)
-			)
-			(justify right)
-		)
-		(property "Intersheetrefs" "${INTERSHEET_REFS}"
-			(at 73.434 106.68 0)
 			(hide yes)
 			(show_name no)
@@
 	)
 	(symbol
+		(lib_id "power:GND")
+		(at 228.6 69.85 0)
+		(unit 1)
+		(body_style 1)
+		(exclude_from_sim no)
+		(in_bom yes)
+		(on_board yes)
+		(in_pos_files yes)
+		(dnp no)
+		(fields_autoplaced yes)
+		(property "Reference" "#PWR010"
+			(at 228.6 76.2 0)
+			(hide yes)
+			(show_name no)
+			(do_not_autoplace no)
+			(effects
+				(font
+					(size 1.27 1.27)
+				)
+			)
+		)
+		(property "Value" "GND"
+			(at 228.6 74.93 0)
+			(show_name no)
+			(do_not_autoplace no)
+			(effects
+				(font
+					(size 1.27 1.27)
+				)
+			)
+		)
+		(property "Footprint" ""
+			(at 228.6 69.85 0)
+			(hide yes)
+			(show_name no)
+			(do_not_autoplace no)
+			(effects
+				(font
+					(size 1.27 1.27)
+				)
+			)
+		)
+		(property "Datasheet" ""
+			(at 228.6 69.85 0)
+			(hide yes)
+			(show_name no)
+			(do_not_autoplace no)
+			(effects
+				(font
+					(size 1.27 1.27)
+				)
+			)
+		)
+		(property "Description" "Power symbol creates a global label with name \"GND\" , ground"
+			(at 228.6 69.85 0)
+			(hide yes)
+			(show_name no)
+			(do_not_autoplace no)
+			(effects
+				(font
+					(size 1.27 1.27)
+				)
+			)
+		)
+		(pin "1"
+		)
+		(instances
+			(project "OsmoFresh_Quella_PRO"
+				(path "/085f93a2-5d2b-46a2-ac0d-b864eaf3f9e9/2b9333e9-34a2-4912-b9d7-bd9dc2d53cb4"
+					(reference "#PWR010")
+					(unit 1)
+				)
+			)
+		)
+	)
+	(symbol
 		(lib_id "Device:C")
 		(at 190.5 63.5 180)
@@
 	)
 	(symbol
+		(lib_id "power:+5V")
+		(at 177.8 55.88 0)
+		(unit 1)
+		(body_style 1)
+		(exclude_from_sim no)
+		(in_bom yes)
+		(on_board yes)
+		(in_pos_files yes)
+		(dnp no)
+		(fields_autoplaced yes)
+		(property "Reference" "#PWR011"
+			(at 177.8 59.69 0)
+			(hide yes)
+			(show_name no)
+			(do_not_autoplace no)
+			(effects
+				(font
+					(size 1.27 1.27)
+				)
+			)
+		)
+		(property "Value" "+5V"
+			(at 177.8 50.8 0)
+			(show_name no)
+			(do_not_autoplace no)
+			(effects
+				(font
+					(size 1.27 1.27)
+				)
+			)
+		)
+		(property "Footprint" ""
+			(at 177.8 55.88 0)
+			(hide yes)
+			(show_name no)
+			(do_not_autoplace no)
+			(effects
+				(font
+					(size 1.27 1.27)
+				)
+			)
+		)
+		(property "Datasheet" ""
+			(at 177.8 55.88 0)
+			(hide yes)
+			(show_name no)
+			(do_not_autoplace no)
+			(effects
+				(font
+					(size 1.27 1.27)
+				)
+			)
+		)
+		(property "Description" "Power symbol creates a global label with name \"+5V\""
+			(at 177.8 55.88 0)
+			(hide yes)
+			(show_name no)
+			(do_not_autoplace no)
+			(effects
+				(font
+					(size 1.27 1.27)
+				)
+			)
+		)
+		(pin "1"
+		)
+		(instances
+			(project "OsmoFresh_Quella_PRO"
+				(path "/085f93a2-5d2b-46a2-ac0d-b864eaf3f9e9/2b9333e9-34a2-4912-b9d7-bd9dc2d53cb4"
+					(reference "#PWR011")
+					(unit 1)
+				)
+			)
+		)
+	)
+	(symbol
 		(lib_id "Device:R")
 		(at 86.36 128.27 90)
@@
 					(unit 1)
 				)
+			)
+		)
+	)
+	(symbol
+		(lib_id "power:GND")
+		(at 140.97 132.08 0)
+		(unit 1)
+		(body_style 1)
+		(exclude_from_sim no)
+		(in_bom yes)
+		(on_board yes)
+		(in_pos_files yes)
+		(dnp no)
+		(fields_autoplaced yes)
+		(property "Reference" "#PWR09"
+			(at 140.97 138.43 0)
+			(hide yes)
+			(show_name no)
+			(do_not_autoplace no)
+			(effects
+				(font
+					(size 1.27 1.27)
+				)
+			)
+		)
+		(property "Value" "GND"
+			(at 140.97 137.16 0)
+			(show_name no)
+			(do_not_autoplace no)
+			(effects
+				(font
+					(size 1.27 1.27)
+				)
+			)
+		)
+		(property "Footprint" ""
+			(at 140.97 132.08 0)
+			(hide yes)
+			(show_name no)
+			(do_not_autoplace no)
+			(effects
+				(font
+					(size 1.27 1.27)
+				)
+			)
+		)
+		(property "Datasheet" ""
+			(at 140.97 132.08 0)
+			(hide yes)
+			(show_name no)
+			(do_not_autoplace no)
+			(effects
+				(font
+					(size 1.27 1.27)
+				)
+			)
+		)
+		(property "Description" "Power symbol creates a global label with name \"GND\" , ground"
+			(at 140.97 132.08 0)
+			(hide yes)
+			(show_name no)
+			(do_not_autoplace no)
+			(effects
+				(font
+					(size 1.27 1.27)
+				)
+			)
+		)
+		(pin "1"
+		)
+		(instances
+			(project "OsmoFresh_Quella_PRO"
+				(path "/085f93a2-5d2b-46a2-ac0d-b864eaf3f9e9/2b9333e9-34a2-4912-b9d7-bd9dc2d53cb4"
+					(reference "#PWR09")
+					(unit 1)
+				)

Commit message: Update Schematics
Parts:
- added CN11: Conn_01x04_Pin, symbol Connector:Conn_01x04_Pin
- added CN6, CN7, CN9: Conn_01x02_Pin, symbol Connector:Conn_01x02_Pin
Connections:
- net +5V: now also CN11.4 (Pin_4)
- net Display_RX: now also CN11.3 (Pin_3)
- net Display_TX: now also CN11.2 (Pin_2)
- net GND: now also CN11.1 (Pin_1)
- net Internal_Tank_Level_Black+: now also CN6.2 (Pin_2)
- net TDS+: now also CN9.1 (Pin_1)
- net TDS-: now also CN9.2 (Pin_2)
- net UNUSED_CN7+: now also CN7.1 (Pin_1)
- net UNUSED_CN7-: now also CN7.2 (Pin_2)
- new net Internal_Tank_Level_Black-: CN6.1 (Pin_1)

Commit message: Update Schematics
Parts:
- renumbered C28 to C22, C29 to C23, C30 to C24, C2 to C25, C17 to C26, C14 to C27, CN6 to CN11, CN7 to CN12, CN11 to CN13, CN9 to CN14, R69 to R47, R13 to R48, R38 to R49, R56 to R50, R57 to R51, R12 to R52, R8 to R53, R46 to R54

Commit message: Update Schematics
Parts:
- renumbered C27 to C14, C26 to C17, C25 to C2, C22 to C28, C23 to C29, C24 to C30, CN13 to CN10, CN11 to CN6, CN12 to CN7, CN14 to CN9, R52 to R12, R48 to R13, R49 to R38, R54 to R46, R50 to R56, R51 to R57, R47 to R69, R53 to R8

Commit message: Update Schematics
Parts:
- removed C28, C29, C30: unkown, symbol Device:C
- removed CN10: Conn_01x04_Pin, symbol Connector:Conn_01x04_Pin
- removed R38, R69, R8: 2kΩ, symbol Device:R
- removed R56, R57: 220Ω, symbol Device:R
- added C23, C24, C25, C26: unkown, symbol Device:C
- added CN11: Conn_01x04_Pin, symbol Connector:Conn_01x04_Pin
- added CN14, CN2: Conn_01x02_Pin, symbol Connector:Conn_01x02_Pin
- added R14, R21: 1kΩ, symbol Device:R
- added R16, R24, R4: 2kΩ, symbol Device:R
- added R49, R50: 220Ω, symbol Device:R
- added R67, R68: 10kΩ, symbol Device:R
Connections:
- net Internal_Tank_Level_Black- is gone; now on an unnamed net: CN6.1 (Pin_1)
- net +5V: now also CN11.1 (Pin_1), R67.1, R68.1
- net Display_RX: now also C23.2, R49.2, R67.2
- net Display_TX: now also C24.2, R50.1, R68.2
- net GND: now also CN6.2 (Pin_2), C23.1, C24.1, CN11.4 (Pin_4), CN14.2 (Pin_2), CN2.1 (Pin_1)
- net Internal_Tank_Level_High_orLow_Black: now reaches R12.1
- net Internal_Tank_Level_High_orLow_Red: now reaches R13.1
- net Internal_Tank_Level_Black+: no longer names the net of R12.2
- net Internal_Tank_Level_Black+: no longer CN6.2 (Pin_2)
- net Internal_Tank_Level_Red+: no longer names the net of R13.2
- net Internal_Tank_Level_Red+: now also CN14.1 (Pin_1)
- net TDS-: no longer names the net of CN9.2 (Pin_2)
- net TDS-: now also C25.2, R21.1, R24.1
- net UNUSED_CN7-: no longer names the net of CN7.2 (Pin_2)
- net UNUSED_CN7-: now also C26.2, R14.1, R16.1
- new net: CN11.2 (Pin_2), R49.1
- new net: CN11.3 (Pin_3), R50.2
- new net: CN2.2 (Pin_2), R4.1
- new net TDS_1: R24.2
- new net TDS_2: C25.1, R21.2
- new net UNUSED_CN7_1: R16.2
- new net UNUSED_CN7_2: C26.1, R14.2
- new net Water_Tank_Empty: R4.2
Other:
- moved on the sheet: C14, C17, C2, R46

Commit message: Update Schematics
Parts:
- removed C14, C17, C2: unkown, symbol Device:C
- removed R46: 330Ω, symbol Device:R
