File: KiCAD/OsmoFresh_Quella_PRO/MainPCB.MCU.kicad_sch (KiCad schematic)
At the start: 21 parts, among them CN11 Conn_01x04_Pin, CN14 Conn_01x02_Pin, CN2 Conn_01x02_Pin, CN6 Conn_01x02_Pin, CN7 Conn_01x02_Pin, CN9 Conn_01x02_Pin

Commit message: Update Schematics
Parts:
- added C13: unkown, symbol Device:C
Connections:
- net +5V: now also C13.2
- net GND: now also C13.1
Other:
- moved on the sheet: C23, C24, CN11, R49, R50, R67, R68

Commit message: Update Schematics
Other:
- note added: "Internel Tank Level"
- note added: "MCU"
- note added: "TDS"
- note added: "UART Userinterface"
- note added: "UNUSED CH7"
- note added: "Water Tank Empty"
- moved on the sheet: C13, C23, C24, C25, C26, CN11, CN14, CN2, CN6, CN7, CN9, R12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

Commit message: Update Documentation
Connections:
- net GND: now also CN14.1 (Pin_1), CN6.1 (Pin_1); no longer CN14.2 (Pin_2), CN6.2 (Pin_2)
- net at R12.2: now also CN6.2 (Pin_2); no longer CN6.1 (Pin_1)
- net at R13.2: now also CN14.2 (Pin_2); no longer CN14.1 (Pin_1)
- net Internal_Tank_Level_High_orLow_Black renamed Internal_Tank_Level_Max
- net Internal_Tank_Level_High_orLow_Red renamed Internal_Tank_Level_Min
Other:
- note added: "Internal Tank Level MAX > 180 mm (100%)"
- note added: "Internal Tank Level MIN > 90 mm (50%)"
- note removed: "Internel Tank Level"
- moved on the sheet: C26, CN14, CN2, CN6, CN7, R12, R13, R14, R16, R4

Commit message: Update Schematics
Other:
- moved on the sheet: CN14, CN6, R12, R13
Changed lines of the file:
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@@
 	(title_block
 		(title "MainPCB MCU")
-		(date "2026-08-20")
+		(date "2026-08-22")
 		(rev "1.0.0")
 		(company "LostCacher")
@@
 	(rectangle
 		(start 25.4 165.1)
-		(end 127 241.3)
+		(end 127 228.6)
 		(stroke
 			(width 0)
@@
 	(rectangle
 		(start 139.7 165.1)
-		(end 241.3 241.3)
+		(end 241.3 228.6)
 		(stroke
 			(width 0)
@@
 	(wire
 		(pts
-			(xy 203.2 203.2) (xy 203.2 190.5)
+			(xy 203.2 190.5) (xy 203.2 177.8)
 		)
 		(stroke
@@
 	(wire
 		(pts
-			(xy 88.9 190.5) (xy 80.01 190.5)
-		)
-		(stroke
-			(width 0)
-			(type default)
-		)
-	)
-	(wire
-		(pts
-			(xy 177.8 177.8) (xy 177.8 187.96)
+			(xy 88.9 177.8) (xy 80.01 177.8)
 		)
 		(stroke
@@
 	(wire
 		(pts
-			(xy 177.8 190.5) (xy 186.69 190.5)
+			(xy 177.8 177.8) (xy 186.69 177.8)
 		)
 		(stroke
@@
 	(wire
 		(pts
-			(xy 88.9 203.2) (xy 88.9 190.5)
+			(xy 88.9 190.5) (xy 88.9 177.8)
 		)
 		(stroke
@@
 	(wire
 		(pts
-			(xy 63.5 190.5) (xy 72.39 190.5)
+			(xy 63.5 177.8) (xy 72.39 177.8)
 		)
 		(stroke
@@
 	(wire
 		(pts
+			(xy 177.8 180.34) (xy 177.8 190.5)
+		)
+		(stroke
+			(width 0)
+			(type default)
+		)
+	)
+	(wire
+		(pts
 			(xy 88.9 73.66) (xy 102.87 73.66)
 		)
@@
 	(wire
 		(pts
-			(xy 292.1 99.06) (xy 292.1 92.71)
+			(xy 63.5 180.34) (xy 63.5 190.5)
 		)
 		(stroke
@@
 	(wire
 		(pts
-			(xy 125.73 85.09) (xy 139.7 85.09)
+			(xy 292.1 99.06) (xy 292.1 92.71)
 		)
 		(stroke
@@
 	(wire
 		(pts
-			(xy 368.3 66.04) (xy 368.3 87.63)
+			(xy 125.73 85.09) (xy 139.7 85.09)
 		)
 		(stroke
@@
 	(wire
 		(pts
-			(xy 279.4 82.55) (xy 279.4 85.09)
+			(xy 368.3 66.04) (xy 368.3 87.63)
 		)
 		(stroke
@@
 	(wire
 		(pts
-			(xy 203.2 190.5) (xy 194.31 190.5)
+			(xy 279.4 82.55) (xy 279.4 85.09)
 		)
 		(stroke
@@
 	(wire
 		(pts
-			(xy 266.7 76.2) (xy 266.7 82.55)
+			(xy 203.2 177.8) (xy 194.31 177.8)
 		)
 		(stroke
@@
 	(wire
 		(pts
-			(xy 63.5 177.8) (xy 63.5 187.96)
+			(xy 266.7 76.2) (xy 266.7 82.55)
 		)
 		(stroke
@@
 	(global_label "Internal_Tank_Level_Min"
 		(shape output)
-		(at 203.2 203.2 270)
+		(at 203.2 190.5 270)
 		(fields_autoplaced yes)
 		(effects
@@
 		)
 		(property "Intersheetrefs" "${INTERSHEET_REFS}"
-			(at 203.2 228.7425 90)
+			(at 203.2 216.0425 90)
 			(hide yes)
 			(show_name no)
@@
 		)
 	)
-	(global_label "IC1_Pin12"
-		(shape bidirectional)
+	(global_label "AC_Sense"
+		(shape input)
 		(at 139.7 58.42 0)
 		(fields_autoplaced yes)
@@
 		)
 		(property "Intersheetrefs" "${INTERSHEET_REFS}"
-			(at 153.2912 58.42 0)
+			(at 151.5752 58.42 0)
 			(hide yes)
 			(show_name no)
@@
 	(global_label "Internal_Tank_Level_Max"
 		(shape output)
-		(at 88.9 203.2 270)
+		(at 88.9 190.5 270)
 		(fields_autoplaced yes)
 		(effects
@@
 		)
 		(property "Intersheetrefs" "${INTERSHEET_REFS}"
-			(at 88.9 229.1658 90)
+			(at 88.9 216.4658 90)
 			(hide yes)
 			(show_name no)
@@
 	(symbol
 		(lib_id "power:GND")
-		(at 177.8 177.8 180)
+		(at 177.8 190.5 0)
 		(unit 1)
 		(body_style 1)
@@
 		(fields_autoplaced yes)
 		(property "Reference" "#PWR032"
-			(at 177.8 171.45 0)
+			(at 177.8 196.85 0)
 			(hide yes)
 			(show_name no)
@@
 		)
 		(property "Value" "GND"
-			(at 180.34 176.5299 0)
+			(at 180.34 191.7699 0)
 			(show_name no)
 			(do_not_autoplace no)
@@
 					(size 1.27 1.27)
 				)
-				(justify right)
+				(justify left)
 			)
 		)
 		(property "Footprint" ""
-			(at 177.8 177.8 0)
+			(at 177.8 190.5 0)
 			(hide yes)
 			(show_name no)
@@
 		)
 		(property "Datasheet" ""
-			(at 177.8 177.8 0)
+			(at 177.8 190.5 0)
 			(hide yes)
 			(show_name no)
@@
 		)
 		(property "Description" "Power symbol creates a global label with name \"GND\" , ground"
-			(at 177.8 177.8 0)
+			(at 177.8 190.5 0)
 			(hide yes)
 			(show_name no)
@@
 	(symbol
 		(lib_id "Device:R")
-		(at 76.2 190.5 270)
+		(at 76.2 177.8 270)
 		(unit 1)
 		(body_style 1)
@@
 		(dnp no)
 		(property "Reference" "R12"
-			(at 76.2 185.928 90)
+			(at 76.2 173.228 90)
 			(show_name no)
 			(do_not_autoplace no)
@@
 		)
 		(property "Value" "2kΩ"
-			(at 76.2 187.96 90)
+			(at 76.2 175.26 90)
 			(show_name no)
 			(do_not_autoplace no)
@@
 		)
 		(property "Footprint" ""
-			(at 76.2 188.722 90)
+			(at 76.2 176.022 90)
 			(hide yes)
 			(show_name no)
@@
 		)
 		(property "Datasheet" ""
-			(at 76.2 190.5 0)
+			(at 76.2 177.8 0)
 			(hide yes)
 			(show_name no)
@@
 		)
 		(property "Description" "Resistor"
-			(at 76.2 190.5 0)
+			(at 76.2 177.8 0)
 			(hide yes)
 			(show_name no)
@@
 	(symbol
 		(lib_id "Device:R")
-		(at 190.5 190.5 270)
+		(at 190.5 177.8 270)
 		(unit 1)
 		(body_style 1)
@@
 		(dnp no)
 		(property "Reference" "R13"
-			(at 190.5 186.182 90)
+			(at 190.5 173.482 90)
 			(show_name no)
 			(do_not_autoplace no)
@@
 		)
 		(property "Value" "2kΩ"
-			(at 190.5 188.214 90)
+			(at 190.5 175.514 90)
 			(show_name no)
 			(do_not_autoplace no)
@@
 		)
 		(property "Footprint" ""
-			(at 190.5 188.722 90)
+			(at 190.5 176.022 90)
 			(hide yes)
 			(show_name no)
@@
 		)
 		(property "Datasheet" ""
-			(at 190.5 190.5 0)
+			(at 190.5 177.8 0)
 			(hide yes)
 			(show_name no)
@@
 		)
 		(property "Description" "Resistor"
-			(at 190.5 190.5 0)
+			(at 190.5 177.8 0)
 			(hide yes)
 			(show_name no)
@@
 	(symbol
 		(lib_id "power:GND")
-		(at 63.5 177.8 180)
+		(at 63.5 190.5 0)
 		(unit 1)
 		(body_style 1)
@@
 		(fields_autoplaced yes)
 		(property "Reference" "#PWR033"
-			(at 63.5 171.45 0)
+			(at 63.5 196.85 0)
 			(hide yes)
 			(show_name no)
@@
 		)
 		(property "Value" "GND"
-			(at 66.04 176.5299 0)
+			(at 66.04 191.7699 0)
 			(show_name no)
 			(do_not_autoplace no)
@@
 					(size 1.27 1.27)
 				)
-				(justify right)
+				(justify left)
 			)
 		)
 		(property "Footprint" ""
-			(at 63.5 177.8 0)
+			(at 63.5 190.5 0)
 			(hide yes)
 			(show_name no)
@@
 		)
 		(property "Datasheet" ""
-			(at 63.5 177.8 0)
+			(at 63.5 190.5 0)
 			(hide yes)
 			(show_name no)
@@
 		)
 		(property "Description" "Power symbol creates a global label with name \"GND\" , ground"
-			(at 63.5 177.8 0)
+			(at 63.5 190.5 0)
 			(hide yes)
 			(show_name no)
@@
 	(symbol
 		(lib_id "Connector:Conn_01x02_Pin")
-		(at 172.72 187.96 0)
+		(at 172.72 180.34 0)
+		(mirror x)
 		(unit 1)
 		(body_style 1)
@@
 		(dnp no)
 		(property "Reference" "CN14"
-			(at 169.926 189.23 0)
+			(at 169.926 179.07 0)
 			(show_name no)
 			(do_not_autoplace no)
@@
 		)
 		(property "Value" "Conn_01x02_Pin"
-			(at 173.355 185.42 0)
+			(at 173.355 182.88 0)
 			(hide yes)
 			(show_name no)
@@
 		)
 		(property "Footprint" ""
-			(at 172.72 187.96 0)
+			(at 172.72 180.34 0)
 			(hide yes)
 			(show_name no)
@@
 		)
 		(property "Datasheet" ""
-			(at 172.72 187.96 0)
+			(at 172.72 180.34 0)
 			(hide yes)
 			(show_name no)
@@
 		)
 		(property "Description" "Generic connector, single row, 01x02, script generated"
-			(at 172.72 187.96 0)
+			(at 172.72 180.34 0)
 			(hide yes)
 			(show_name no)
@@
 	(symbol
 		(lib_id "Connector:Conn_01x02_Pin")
-		(at 58.42 187.96 0)
+		(at 58.42 180.34 0)
+		(mirror x)
 		(unit 1)
 		(body_style 1)
@@
 		(dnp no)
 		(property "Reference" "CN6"
-			(at 55.118 189.23 0)
+			(at 55.118 179.07 0)
 			(show_name no)
 			(do_not_autoplace no)
@@
 		)
 		(property "Value" "Conn_01x02_Pin"
-			(at 59.055 185.42 0)
+			(at 59.055 182.88 0)
 			(hide yes)
 			(show_name no)
@@
 		)
 		(property "Footprint" ""
-			(at 58.42 187.96 0)
+			(at 58.42 180.34 0)
 			(hide yes)
 			(show_name no)
@@
 		)
 		(property "Datasheet" ""
-			(at 58.42 187.96 0)
+			(at 58.42 180.34 0)
 			(hide yes)
 			(show_name no)
@@
 		)
 		(property "Description" "Generic connector, single row, 01x02, script generated"
-			(at 58.42 187.96 0)
+			(at 58.42 180.34 0)
 			(hide yes)
 			(show_name no)

Commit message: Update Schematics
Other:
- note added: "UART (Display)"
- note removed: "UART Userinterface"
Changed lines of the file:
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@@
 		)
 	)
-	(text "UART Userinterface"
+	(text "UART (Display)"
 		(exclude_from_sim no)
 		(at 266.7 33.02 0)
