File: KiCAD/OsmoFresh_Quella_PRO/MainPCB.24Vdc.kicad_sch (KiCad schematic)
At the start: 67 parts, among them CN1 Conn_01x02_Pin, CN10 Conn_01x06_Pin, CN12 Conn_01x02_Pin, CN13 Conn_01x02_Pin, K2 5A 250Vac, Q2 NMOS, Q3 NPN, Q4 PMOS, Q5 NPN, Q6 NPN, Q8 NPN, U4 ULN2003A

Commit message: Update Schematics
Parts:
- renumbered C25 to C1, C12 to C10, C6 to C11, C1 to C12, C4 to C13, C19 to C14, C18 to C15, C5 to C2, C20 to C3, C7 to C4, C16 to C5, C8 to C6, C15 to C7, C9 to C8, C13 to C9, CN13 to CN1, CN12 to CN2, CN10 to CN3, CN1 to CN4, D5 to D1, D7 to D2, D6 to D3, Q5 to Q2, Q6 to Q3, Q3 to Q4, Q8 to Q5, Q4 to Q6, Q2 to Q7, R60 to R1, R67 to R10, R23 to R11, R16 to R12, R68 to R13, R21 to R14, R18 to R15, R20 to R16, R19 to R17, R34 to R18, R39 to R19, R59 to R2, R64 to R20, R62 to R21, R63 to R22, R37 to R23, R35 to R24, R36 to R25, R32 to R29, R10 to R3, R33 to R30, R6 to R31, R17 to R32, R51 to R33, R52 to R34, R5 to R35, R15 to R36, R55 to R37, R53 to R38, R54 to R39, R61 to R4, R11 to R5, R66 to R6, R31 to R8, R14 to R9, U4 to U1

Commit message: Update Schematics
Parts:
- removed C10, C3, C4, C6, C8, C9: unkown, symbol Device:C
- removed Q3, Q4: NPN, symbol Simulation_SPICE:NPN
- removed R1, R16: 10kΩ, symbol Device:R
- removed R11, R4: 47kΩ, symbol Device:R
- removed R15, R8: 4,7kΩ, symbol Device:R
- removed R17, R2: 470Ω, symbol Device:R
- renumbered C12 to C1, C7 to C12, C5 to C13, C15 to C18, C14 to C19, C1 to C25, C13 to C4, C2 to C5, C11 to C6, CN4 to CN1, CN3 to CN10, CN2 to CN12, CN1 to CN13, D1 to D5, D3 to D6, D2 to D7, Q7 to Q2, Q6 to Q4, Q2 to Q5, Q5 to Q8, R3 to R10, R5 to R11, R9 to R14, R36 to R15, R12 to R16, R32 to R17, R14 to R21, R29 to R32, R30 to R33, R18 to R34, R24 to R35, R25 to R36, R23 to R37, R19 to R39, R35 to R5, R33 to R51, R34 to R52, R38 to R53, R39 to R54, R37 to R55, R31 to R6, R21 to R62, R22 to R63, R20 to R64, R6 to R66, R10 to R67, R13 to R68, U1 to U4
Other:
- moved on the sheet: C12, C13, C25, C5, R10, R11, R14, R16, R21, R66, R67, R68

Commit message: Update Schematics
Parts:
- removed C25, C4, C5: unkown, symbol Device:C
- removed R10, R5, R66: 2kΩ, symbol Device:R
- removed R11, R6, R67, R68: 10kΩ, symbol Device:R
- removed R14, R16, R21: 1kΩ, symbol Device:R

Commit message: Update Schematics
Parts:
- removed C12, C13: unkown, symbol Device:C
Connections:
- net GND: now also R35.2, R36.2, R37.2; no longer U4.8 (GND)
- net Water_Pump-: now also R64.1; no longer R35.2, R37.2
- net IC1_Pin16 renamed Water_Pump_Current
Other:
- moved on the sheet: C18, C19, D4, D6, Q2, Q4, Q8, R15, R17, R32, R33, R51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

Commit message: Update Schematics
Parts:
- added C12: unkown, symbol Device:C
- R32: value 5,1kΩ -> 510Ω
- R35, R36, R37: value 20kΩ -> 10kΩ
- renumbered R39 to R38
Connections:
- net +24V: now also C12.2
- net GND: now also C12.1
Changed lines of the file:
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@@
 	)
 	(junction
+		(at 391.16 508)
+		(diameter 0)
+		(color 0 0 0 0)
+	)
+	(junction
 		(at 441.96 532.13)
 		(diameter 0)
@@
 	(wire
 		(pts
+			(xy 412.75 508) (xy 391.16 508)
+		)
+		(stroke
+			(width 0)
+			(type default)
+		)
+	)
+	(wire
+		(pts
 			(xy 478.79 355.6) (xy 483.87 355.6)
 		)
@@
 	(wire
 		(pts
+			(xy 391.16 325.12) (xy 391.16 508)
+		)
+		(stroke
+			(width 0)
+			(type default)
+		)
+	)
+	(wire
+		(pts
 			(xy 391.16 519.43) (xy 412.75 519.43)
 		)
@@
 	(wire
 		(pts
+			(xy 391.16 508) (xy 391.16 519.43)
+		)
+		(stroke
+			(width 0)
+			(type default)
+		)
+	)
+	(wire
+		(pts
 			(xy 516.89 342.9) (xy 516.89 345.44)
 		)
@@
 	(wire
 		(pts
-			(xy 534.67 431.8) (xy 538.48 431.8)
+			(xy 420.37 508) (xy 441.96 508)
 		)
 		(stroke
@@
 	(wire
 		(pts
-			(xy 391.16 325.12) (xy 391.16 519.43)
+			(xy 534.67 431.8) (xy 538.48 431.8)
 		)
 		(stroke
@@
 		(in_pos_files yes)
 		(dnp no)
-		(property "Reference" "R39"
+		(property "Reference" "R38"
 			(at 377.19 273.05 90)
 			(show_name no)
@@
 			(project "OsmoFresh_Quella_PRO"
 				(path "/4260df0e-d900-46a1-97d3-cde6b2933985/00785b84-3607-4d80-92ae-17ec4beff254"
-					(reference "R39")
+					(reference "R38")
 					(unit 1)
 				)
@@
 	)
 	(symbol
+		(lib_id "Device:C")
+		(at 416.56 508 270)
+		(unit 1)
+		(body_style 1)
+		(exclude_from_sim no)
+		(in_bom yes)
+		(on_board yes)
+		(in_pos_files yes)
+		(dnp no)
+		(property "Reference" "C12"
+			(at 416.56 504.698 90)
+			(show_name no)
+			(do_not_autoplace no)
+			(effects
+				(font
+					(size 1.27 1.27)
+				)
+			)
+		)
+		(property "Value" "unkown"
+			(at 416.56 511.556 90)
+			(hide yes)
+			(show_name no)
+			(do_not_autoplace no)
+			(effects
+				(font
+					(size 1.27 1.27)
+				)
+			)
+		)
+		(property "Footprint" ""
+			(at 412.75 508.9652 0)
+			(hide yes)
+			(show_name no)
+			(do_not_autoplace no)
+			(effects
+				(font
+					(size 1.27 1.27)
+				)
+			)
+		)
+		(property "Datasheet" ""
+			(at 416.56 508 0)
+			(hide yes)
+			(show_name no)
+			(do_not_autoplace no)
+			(effects
+				(font
+					(size 1.27 1.27)
+				)
+			)
+		)
+		(property "Description" "Unpolarized capacitor"
+			(at 416.56 508 0)
+			(hide yes)
+			(show_name no)
+			(do_not_autoplace no)
+			(effects
+				(font
+					(size 1.27 1.27)
+				)
+			)
+		)
+		(pin "2"
+		)
+		(pin "1"
+		)
+		(instances
+			(project "OsmoFresh_Quella_PRO"
+				(path "/4260df0e-d900-46a1-97d3-cde6b2933985/00785b84-3607-4d80-92ae-17ec4beff254"
+					(reference "C12")
+					(unit 1)
+				)
+			)
+		)
+	)
+	(symbol
 		(lib_id "Device:R")
 		(at 480.06 406.4 180)
@@
 			)
 		)
-		(property "Value" "5,1kΩ"
+		(property "Value" "510Ω"
 			(at 484.886 407.67 0)
 			(show_name no)
@@
 			)
 		)
-		(property "Value" "20kΩ"
+		(property "Value" "10kΩ"
 			(at 454.66 342.9 90)
 			(show_name no)
@@
 			)
 		)
-		(property "Value" "20kΩ"
+		(property "Value" "10kΩ"
 			(at 454.406 332.994 90)
 			(show_name no)
@@
 			)
 		)
-		(property "Value" "20kΩ"
+		(property "Value" "10kΩ"
 			(at 454.66 353.06 90)
 			(show_name no)

Commit message: Update Schematics
Parts:
- removed CN13: Conn_01x02_Pin, symbol Connector:Conn_01x02_Pin
- added K1: 10A 250Vac, symbol Relay:Relay_SPST-NO
Connections:
- net +24V: now also K1.A1
- net GND: now also C18.1, C19.1, Q2.3 (S), R33.1, R38.2; no longer Q2.1 (D)
- net at Q8.2 (B): now also R32.1, R33.2; no longer R33.1
- net at R34.2, R38.1: now also Q5.2 (B)
- net Feed_Pump_Current: now reaches C18.2
- net Feed_Pump_Current: now also R54.2; no longer C19.1
- net at R15.1, R17.1: now also Q2.2 (G); no longer Q2.3 (S)
- net Heat_1200W renamed Heater_1200W_Enable
- removed net IC1_Pin15: C18.1, R54.2
- net IC1_Pin3 renamed Feed_Pump_Enable
- net IC1_Pin5 renamed Flush_Valve_Enable
- net IC1_Pin6 renamed UNUSED_CH10_Enable
- net IC1_Pin7 renamed UNUSED_CH13_Enable
- net K2_Water_Pump renamed Booster_Pump_Enable
- net Relay_Heater_Coil-: no longer names the net of D4.2 (A)
- net Relay_Heater_Coil-: now also Q2.1 (D), K1.A2; no longer Q2.2 (G)
- net Water_Outlet_Valve+: no longer names the net of CN12.1 (Pin_1), D6.1 (K), Q4.1 (D)
- net Water_Outlet_Valve-: no longer names the net of CN12.2 (Pin_2), D6.2 (A), R53.1, R55.2
- net Water_Pump+ renamed Booster_Pump+
- net Water_Pump- renamed Booster_Pump-
- net Water_Pump_Current renamed Booster_Pump_Current
- new net Heater_1200W: K1.14
- new net LINE: K1.13
Other:
- note added: "+24 Vdc Power Supply"
- note added: "Booster Pump + Current"
- note added: "CN10 Connection"
- note added: "Feed Pump + Current"
- note added: "Heat 1200 Watt"
- note added: "P2"
- note added: "Valve Control"
- note added: "Vuanze Electric Y32F-SS-124HM"
- moved on the sheet: C1, C12, C6, CN1, CN10, D5, D7, EC1, Q5, R34, R35, R36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
