File: KiCAD/OsmoFresh_Quella_PRO/MainPCB.5Vdc.kicad_sch (KiCad schematic)
At the start: 17 parts, among them U5 KM393

Commit message: Update Schematics
Parts:
- added CN14, CN16, CN2, CN3, CN5, CN8: Conn_01x02_Pin, symbol Connector:Conn_01x02_Pin
Connections:
- new net Internal_Tank_Level_Red+: CN14.2 (Pin_2)
- new net Internal_Tank_Level_Red-: CN14.1 (Pin_1)
- new net Temperature_Inlet+: CN5.1 (Pin_1)
- new net Temperature_Inlet-: CN5.2 (Pin_2)
- new net Temperature_Outlet+: CN3.1 (Pin_1)
- new net Temperature_Outlet-: CN3.2 (Pin_2)
- new net UNUSED_CN16+: CN16.1 (Pin_1)
- new net UNUSED_CN16-: CN16.2 (Pin_2)
- new net UNUSED_CN8+: CN8.1 (Pin_1)
- new net UNUSED_CN8-: CN8.2 (Pin_2)
- new net Water_Tank_Empty+: CN2.1 (Pin_1)
- new net Water_Tank_Empty-: CN2.2 (Pin_2)
Other:
- moved on the sheet: C10, C11, C27, C3, R22, R25, R29, R30, R40, R41, R45, U5

Commit message: Update Schematics
Parts:
- renumbered C22 to C16, C21 to C17, C10 to C18, C27 to C19, C3 to C20, C11 to C21, CN16 to CN10, CN3 to CN5, CN8 to CN6, CN2 to CN7, CN5 to CN8, CN14 to CN9, R29 to R40, R30 to R41, R41 to R42, R40 to R43, R25 to R44, R22 to R46, U5 to U2

Commit message: Update Schematics
Parts:
- removed CN10: Conn_01x02_Pin, symbol Connector:Conn_01x02_Pin
- added C15, C16, C20, C7, C8, C9: unkown, symbol Device:C
- added CN16: Conn_01x02_Pin, symbol Connector:Conn_01x02_Pin
- added Q3, Q6: NPN, symbol Simulation_SPICE:NPN
- added R18, R31: 4,7kΩ, symbol Device:R
- added R19, R59: 470Ω, symbol Device:R
- added R20, R60: 10kΩ, symbol Device:R
- added R23, R61: 47kΩ, symbol Device:R
- renumbered C18 to C10, C21 to C11, C17 to C21, C16 to C22, C19 to C27, C20 to C3, CN9 to CN14, CN7 to CN2, CN5 to CN3, CN8 to CN5, CN6 to CN8, R46 to R22, R44 to R25, R40 to R29, R41 to R30, R43 to R40, R42 to R41, U2 to U5
Connections:
- net UNUSED_CN8+ is gone; now on net +5V: CN8.1 (Pin_1)
- net Water_Tank_Empty- is gone; now on net GND: CN2.2 (Pin_2)
- net +5V: now also C15.2, C7.2, CN16.1 (Pin_1), R18.1, R31.1
- net GND: now also C11.2, C27.1, C3.2, R29.1, R40.2, C16.1, C20.1, C8.1, C9.1, Q3.3 (E), Q6.3 (E), R23.2, R61.2
- net UNUSED_CN8-: no longer names the net of CN8.2 (Pin_2)
- net UNUSED_CN8-: now also C7.1, C9.2, R20.1
- new net: Q3.1 (C), R18.2, R19.1
- new net: Q6.1 (C), R31.2, R59.1
- new net: Q6.2 (B), R60.2, R61.1
- new net: C15.1, C20.2, CN16.2 (Pin_2), R60.1
- new net: Q3.2 (B), R20.2, R23.1
- new net UNUSED_CN16: C16.2, R59.2
- new net UNUSED_CN8: C8.2, R19.2
Other:
- note added: "UNUSED"
- moved on the sheet: C10, C11, C27, C3, CN8, R22, R25, R29, R30, R40, R41, R45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

Commit message: Update Schematics
Parts:
- removed CN14, CN2: Conn_01x02_Pin, symbol Connector:Conn_01x02_Pin
- added C4, C5: unkown, symbol Device:C
- added R10, R5, R65, R66: 2kΩ, symbol Device:R
- added R11, R6: 10kΩ, symbol Device:R
Connections:
- net +5V: now also R65.1, R66.1
- net GND: now also C4.2, C5.1, R11.2, R6.1
- net Temperature_Inlet+: no longer names the net of CN5.1 (Pin_1)
- net Temperature_Inlet+: now also R10.1, R11.1
- net Temperature_Inlet-: no longer names the net of CN5.2 (Pin_2)
- net Temperature_Inlet-: now also R66.2
- net Temperature_Outlet+: no longer names the net of CN3.1 (Pin_1)
- net Temperature_Outlet+: now also R5.2, R6.2
- net Temperature_Outlet-: no longer names the net of CN3.2 (Pin_2)
- net Temperature_Outlet-: now also R65.2
- new net Temperature_Inlet: C5.2, R10.2
- new net Temperature_Outlet: C4.1, R5.1
Other:
- note removed: "UNUSED"
- moved on the sheet: C21, C22, EC2, L1, RL1

Commit message: Update Schematics
Parts:
- added C12, C13, C14, C17, C2: unkown, symbol Device:C
- EC2: value 30µF 10V -> 330µF 10V
Connections:
- net +5V: now also C14.2, C17.2, C2.2
- net GND: now also C14.1, C17.1, C2.1
- net Temperature_Outlet-: now reaches CN3.1 (Pin_1), R5.2, R6.2
- net Temperature_Outlet+: now reaches CN3.2 (Pin_2), R65.2

Commit message: Update Schematics
Parts:
- removed C12, C13: unkown, symbol Device:C
- added U2: VJPN4, Package_TO_SOT_SMD:TSOT-23-5, symbol Regulator_Switching:LM3670MF
Connections:
- net +24V: now also C21.1, U2.1 (Vin); no longer C21.2
- net +5V: now also U2.4 (FB); no longer C14.2, C17.2, C2.2
- net GND: now also C14.2, C17.2, C2.2, C21.2, C22.1, EC2.2, U2.2 (GND); no longer C14.1, C17.1, C2.1
- net at L1.1: now also U2.5 (SW)
- net +5V_MCU: now reaches RL1.2
- net +5V_MCU: now also C14.1, C17.1, C2.1
Other:
- note added: "+5 Vdc Power Supply"
- note removed: "U1 VJPN4"
- moved on the sheet: C10, C15, C16, C20, C27, C3, C4, C5, C7, C8, C9, CN16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

Commit message: Update Schematics
Parts:
- added R44: 330Ω, symbol Device:R
- added R7: 180Ω, symbol Device:R
- added U3: MOC3063M, symbol Relay_SolidState:MOC3063M
- renumbered U2 to U1
Connections:
- net +5V: now also U3.1
- net IC1_Pin11 renamed Zero_Cross_Detected
- new net: R7.1, U3.6
- new net: R44.1, U3.2
- new net Heater_900W_Enable: R44.2
- new net Heater_Triac_Gate: U3.4
- new net LINE: R7.2
Other:
- note added: "Heat 900 Watt"
- note added: "UNUSED CN16"
- note added: "UNUSED CN8"
- note added: "Water Temperature Inlet"
- note added: "Water Temperature Outlet"
- note added: "Zero Cross Dedection"
- moved on the sheet: C10, C11, C14, C15, C16, C17, C2, C20, C21, C22, C27, C3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

Commit message: Update Schematics
Connections:
- net IC1_Pin12 renamed AC_Sense
Changed lines of the file:
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@@
 	(title_block
 		(title "MainPCB +5Vdc")
-		(date "2026-08-20")
+		(date "2026-08-22")
 		(rev "1.0.0")
 		(company "LostCacher")
@@
 		)
 	)
-	(global_label "IC1_Pin12"
-		(shape bidirectional)
+	(global_label "AC_Sense"
+		(shape output)
 		(at 190.5 317.5 0)
 		(fields_autoplaced yes)
@@
 		)
 		(property "Intersheetrefs" "${INTERSHEET_REFS}"
-			(at 204.0912 317.5 0)
+			(at 202.3752 317.5 0)
 			(hide yes)
 			(show_name no)
