File: KiCAD/OsmoFresh_Quella_PRO/MainPCB.5Vdc.kicad_sch (KiCad schematic)
At the start: 52 parts, among them CN16 Conn_01x02_Pin, CN3 Conn_01x02_Pin, CN5 Conn_01x02_Pin, CN8 Conn_01x02_Pin, Q3 NPN, Q6 NPN, U1 VJPN4, U3 MOC3063M, U5 KM393

Commit message: Update Schematics
Other:
- note added: "Zero Cross Detection"
- note removed: "Zero Cross Dedection"
Changed lines of the file:
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@@
 		)
 	)
-	(text "Zero Cross Dedection"
+	(text "Zero Cross Detection"
 		(exclude_from_sim no)
 		(at 133.35 185.42 0)
